Commit message: Implement pickup

File: src/test_bot_controller/urdf/robot_core.xacro (robot description, xacro)
@@ -50,5 +50,5 @@
     <link name="track_1">
         <visual>
-            <origin xyz="0 0 0.09" rpy="${pi/2} 0 ${pi/2}"/>
+            <origin xyz="0 0 0.1" rpy="${pi/2} 0 ${pi/2}"/>
             <geometry>
                 <box size="${track_width} ${track_length} ${track_depth}"/>
@@ -66,8 +66,9 @@
         </xacro:inertial_box>
     </link>
-    <joint name="track1_joint" type="prismatic">
+    <joint name="track1_joint" type="fixed">
         <parent link="chassis"/>
         <child link="track_1"/>
-        <origin xyz="${base_width/2 + track_depth/2} ${base_width/2 - track_width} 0" rpy="0 0 0 " />
+        <!---${base_width/2 - track_width}-->
+        <origin xyz="${base_width/2 + track_depth/2} 0.10 0" rpy="0 0 0" />
         <axis xyz="0 0 1"/>
         <limit effort="110" lower="0" upper="0.6" velocity="0.5"/>
@@ -75,5 +76,5 @@
     <link name="track_2">
         <visual>
-            <origin xyz="0 0 ${track_length/2 - base_height/2}" rpy="${pi/2} 0 ${pi/2}"/>
+            <origin xyz="0 0 0.1" rpy="${pi/2} 0 ${pi/2}"/>
             <geometry>
                 <box size="${track_width} ${track_length} ${track_depth}"/>
@@ -91,8 +92,9 @@
         </xacro:inertial_box>
     </link>
-    <joint name="track2_joint" type="prismatic">
+    <joint name="track2_joint" type="fixed">
         <parent link="chassis"/>
         <child link="track_2"/>
-        <origin xyz="${base_width/2 + track_depth/2} -${base_width/2 - track_width} 0" rpy="0 0 0" />
+        <!---${base_width/2 - track_width}-->
+        <origin xyz="${base_width/2 + track_depth/2} -0.10 0" rpy="0 0 0" />
         <axis xyz="0 0 1"/>
         <limit effort="110" lower="0" upper="0.6" velocity="0.5"/>
@@ -100,14 +102,14 @@
     <link name="fork_plate">
         <visual>
-            <origin xyz="0.0 0 0" rpy="0 0 0"/>
+            <origin xyz="${track_depth} 0.1 0" rpy="0 -${pi/2} 0"/>
+            <geometry>
+                <box size="0.1 0.25 0.02"/>
+            </geometry>
+            <material name="blue"/>
+        </visual>
+        <collision>
+            <origin xyz="0.2 0 0" rpy="0 0 0"/>
             <geometry>
                 <box size="0.5 0.25 0.02"/>
-            </geometry>
-            <material name="blue"/>
-        </visual>
-        <collision>
-            <origin xyz="0 0 0" rpy="0 0 0"/>
-            <geometry>
-                <box size="0.5 0.25 0.2"/>
             </geometry>
         </collision>
@@ -120,5 +122,57 @@
         <child link="fork_plate"/>
         <!--Offset the joint position by the track depth amount-->
-        <origin xyz="0.3 0 0" rpy="0 0 0" />
+        <origin xyz="0 0 0" rpy="0 0 0" />
+        <axis xyz="0 0 1"/>
+        <limit effort="110" lower="0" upper="0.6" velocity="0.5"/>
+    </joint>
+    <link name="fork_1">
+        <visual>
+            <origin xyz="0 0 0" rpy="0 0 -${pi/2}"/>
+            <geometry>
+                <box size="0.05 0.3 0.02"/>
+            </geometry>
+            <material name="white"/>
+        </visual>
+        <collision>
+            <origin xyz="0 0 0" rpy="0 0 -${pi/2}"/>
+            <geometry>
+                <box size="0.5 0.25 0.02"/>
+            </geometry>
+        </collision>
+        <xacro:inertial_box mass="10" x="0" y="0" z="0">
+            <origin xyz="0 0 0" rpy="0 0 -${pi/2}"/>
+        </xacro:inertial_box>
+    </link>
+    <joint name="fork_1_joint" type="fixed">
+        <parent link="fork_plate"/>
+        <child link="fork_1"/>
+        <!--Offset the joint position by the track depth amount-->
+        <origin xyz="0.154 0.05 0" rpy="0 0 0" />
+        <axis xyz="0 0 1"/>
+        <limit effort="110" lower="0" upper="0.6" velocity="0.5"/>
+    </joint>
+    <link name="fork_2">
+        <visual>
+            <origin xyz="0 0 0" rpy="0 0 -${pi/2}"/>
+            <geometry>
+                <box size="0.05 0.3 0.02"/>
+            </geometry>
+            <material name="white"/>
+        </visual>
+        <collision>
+            <origin xyz="0 0 0" rpy="0 0 -${pi/2}"/>
+            <geometry>
+                <box size="0.5 0.25 0.02"/>
+            </geometry>
+        </collision>
+        <xacro:inertial_box mass="10" x="0" y="0" z="0">
+            <origin xyz="0 0 0" rpy="0 0 -${pi/2}"/>
+        </xacro:inertial_box>
+    </link>
+    <joint name="fork_2_joint" type="fixed">
+        <parent link="fork_plate"/>
+        <child link="fork_2"/>
+        <!--Offset the joint position by the track depth amount-->
+        <origin xyz="0.154 0.15 0" rpy="0 0 0" />
         <axis xyz="0 0 1"/>
         <limit effort="110" lower="0" upper="0.6" velocity="0.5"/>
@@ -150,21 +204,23 @@
         <parent link="chassis"/>
         <child link="left_wheel_back"/>
-        <origin xyz="-0.10 0.155 -0.075" rpy="-${pi/2} 0 0" />
-        <axis xyz="0 0 1"/>
+        <origin xyz="-0.10 0.155 -0.075" rpy="0 0 0" />
+        <axis xyz="0 1 0"/>
     </joint>
     <link name="left_wheel_back">
         <visual>
-            <geometry>
-                <cylinder radius="0.05" length="0.02"/>
-            </geometry>
-            <material name="blue"/>
-        </visual>
-        <collision>
-            <geometry>
-                <cylinder radius="0.05" length="0.02"/>
-            </geometry>
-        </collision>
-        <xacro:inertial_cylinder mass="0.1" length="0.02" radius="0.05">
-            <origin xyz="0 0 0" rpy="0 0 0"/>
+            <origin xyz="0 0 0" rpy="0 0 -${pi/2}"/>
+            <geometry>
+                <mesh filename="$(find test_bot_controller)/meshes/flift_wheel.dae" scale="0.0027 0.0027 0.0027"/>
+                <!-- <cylinder radius="0.05" length="0.02"/> -->
+            </geometry>
+        </visual>
+        <collision>
+            <origin xyz="0 0 0" rpy="-${pi/2} 0 0"/>
+            <geometry>
+                <cylinder radius="0.05" length="0.02"/>
+            </geometry>
+        </collision>
+        <xacro:inertial_cylinder mass="0.1" length="0.02" radius="0.05">
+            <origin xyz="0 0 0" rpy="-${pi/2} 0 0"/>
         </xacro:inertial_cylinder>
     </link>
