Commit message: Implement pickup

File: src/test_bot_controller/urdf/robot.urdf.xacro (robot description, xacro)
@@ -21,7 +21,35 @@
             <odom_frame>base_link</odom_frame>
         </plugin>
+        <plugin
+        filename="gz-sim-odometry-publisher-system"
+        name="gz::sim::systems::OdometryPublisher">
+            <odom_frame>base_link</odom_frame>
+            <robot_base_frame>left_wheel</robot_base_frame>
+            <odom_topic>test</odom_topic>
+        </plugin>
+        <plugin filename="gz-sim-odometry-publisher-system" name="gz::sim::systems::OdometryPublisher" >
+            <odom_frame>world</odom_frame>
+            <robot_base_frame>forklift/left_wheel</robot_base_frame>
+            <odom_publish_frequency>10</odom_publish_frequency>
+            <odom_topic>/model/forklift/left_wheel/odometry</odom_topic>
+          </plugin>
+        <!--
+        <plugin
+            filename="gz-sim-pose-publisher-system"
+            name="gz::sim::systems::PosePublisher">
+            <publish_link_pose>true</publish_link_pose>
+            <publish_collision_pose>false</publish_collision_pose>
+            <publish_visual_pose>false</publish_visual_pose>
+            <publish_nested_model_pose>true</publish_nested_model_pose>
+        </plugin>
+        -->
       <plugin filename="gz-sim-joint-state-publisher-system" name="gz::sim::systems::JointStatePublisher">
           <topic>joint_states</topic>
       </plugin>
+      <plugin filename="gz-sim-joint-position-controller-system" name="gz::sim::systems::JointPositionController">
+        <joint_name>fork_plate_joint</joint_name>
+        <topic>fork_control</topic>
+        <initial_position>0.6</initial_position>
+      </plugin>
     </gazebo>
 </robot>

File: src/test_bot_controller/urdf/robot_core.xacro (robot description, xacro)
@@ -15,4 +15,9 @@
     </material>
     <!-- BASE LINK -->
+    <xacro:property name="track_length" value="0.3"/>
+    <xacro:property name="track_depth" value="0.02"/> <!--This is actually the depth of the track when in up position-->
+    <xacro:property name="track_width" value="0.05"/> <!--This is actually the depth of the track when in up position-->
+    <xacro:property name="base_height" value="0.15"/>
+    <xacro:property name="base_width" value="0.3"/>
     <link name="base_link">
     </link>
@@ -27,5 +32,5 @@
             <origin xyz="0 0 0"/>
             <geometry>
-                <box size="0.3 0.3 0.15"/>
+                <box size="0.3 ${base_width} ${base_height}"/>
             </geometry>
             <material name="white"/>
@@ -34,11 +39,83 @@
             <origin xyz="0 0 0"/>
             <geometry>
-                <box size="0.3 0.3 0.15"/>
-            </geometry>
-        </collision>
-        <xacro:inertial_box mass="0.5" x="0.3" y="0.3" z="0.15">
-            <origin xyz="0 0 0" rpy="0 0 0"/>
-        </xacro:inertial_box>
-    </link>
+                <box size="0.3 ${base_width} ${base_height}"/>
+            </geometry>
+        </collision>
+        <xacro:inertial_box mass="500" x="0.3" y="${base_width}" z="${base_height}">
+            <origin xyz="0 0 0" rpy="0 0 0"/>
+        </xacro:inertial_box>
+    </link>
+    <link name="track_1">
+        <visual>
+            <origin xyz="0 0 ${track_length/2 - base_height/2}" rpy="${pi/2} 0 ${pi/2}"/>
+            <geometry>
+                <box size="${track_width} ${track_length} ${track_depth}"/>
+            </geometry>
+            <material name="blue"/>
+        </visual>
+        <collision>
+            <origin xyz="0 0 ${track_length/2 - base_height/2}" rpy="${pi/2} 0 ${pi/2}"/>
+            <geometry>
+                <box size="${track_width} ${track_length} ${track_depth}"/>
+            </geometry>
+        </collision>
+        <xacro:inertial_box mass="10" x="${track_width}" y="${track_length}" z="${track_depth}">
+            <origin xyz="0 0 ${track_length/2 - base_height/2}" rpy="${pi/2} 0 ${pi/2}"/>
+        </xacro:inertial_box>
+    </link>
+    <joint name="track1_joint" type="fixed">
+        <parent link="chassis"/>
+        <child link="track_1"/>
+        <origin xyz="${base_width/2 + track_depth/2} ${base_width/2 - track_width} 0" rpy="0 0 0 " />
+    </joint>
+    <link name="track_2">
+        <visual>
+            <origin xyz="0 0 ${track_length/2 - base_height/2}" rpy="${pi/2} 0 ${pi/2}"/>
+            <geometry>
+                <box size="${track_width} ${track_length} ${track_depth}"/>
+            </geometry>
+            <material name="blue"/>
+        </visual>
+        <collision>
+            <origin xyz="0 0 ${track_length/2 - base_height/2}" rpy="${pi/2} 0 ${pi/2}"/>
+            <geometry>
+                <box size="${track_width} ${track_length} ${track_depth}"/>
+            </geometry>
+        </collision>
+        <xacro:inertial_box mass="10" x="${track_width}" y="${track_length}" z="${track_depth}">
+            <origin xyz="0 0 ${track_length/2 - base_height/2}" rpy="${pi/2} 0 ${pi/2}"/>
+        </xacro:inertial_box>
+    </link>
+    <joint name="track2_joint" type="fixed">
+        <parent link="chassis"/>
+        <child link="track_2"/>
+        <origin xyz="${base_width/2 + track_depth/2} -${base_width/2 - track_width} 0" rpy="0 0 0" />
+    </joint>
+    <link name="fork_plate">
+        <visual>
+            <origin xyz="${track_depth/2} 0.1 0" rpy="0 ${pi/2} 0"/>
+            <geometry>
+                <box size="0.1 0.25 ${track_depth}"/>
+            </geometry>
+            <material name="blue"/>
+        </visual>
+        <collision>
+            <origin xyz="${track_depth/2} 0.1 0" rpy="0 ${pi/2} 0"/>
+            <geometry>
+                <box size="0.1 0.25 ${track_depth}"/>
+            </geometry>
+        </collision>
+        <xacro:inertial_box mass="10" x="0.1" y="0.25" z="${track_depth}">
+            <origin xyz="${track_depth/2} 0.1 0" rpy="0 ${pi/2} 0"/>
+        </xacro:inertial_box>
+    </link>
+    <joint name="fork_plate_joint" type="prismatic">
+        <parent link="track_2"/>
+        <child link="fork_plate"/>
+        <!--Offset the joint position by the track depth amount-->
+        <origin xyz="${track_depth/2} 0 -0.025" rpy="0 0 0" />
+        <axis xyz="0 0 1"/>
+        <limit effort="110" lower="0" upper="0.6" velocity="0.5"/>
+    </joint>
     <!-- LEFT WHEEL LINK -->
     <joint name="left_wheel_joint" type="continuous">

Commit message: Improve pickup

File: src/test_bot_controller/urdf/robot.urdf.xacro (robot description, xacro)
@@ -22,18 +22,4 @@
         </plugin>
         <plugin
-        filename="gz-sim-odometry-publisher-system"
-        name="gz::sim::systems::OdometryPublisher">
-            <odom_frame>base_link</odom_frame>
-            <robot_base_frame>left_wheel</robot_base_frame>
-            <odom_topic>test</odom_topic>
-        </plugin>
-        <plugin filename="gz-sim-odometry-publisher-system" name="gz::sim::systems::OdometryPublisher" >
-            <odom_frame>world</odom_frame>
-            <robot_base_frame>forklift/left_wheel</robot_base_frame>
-            <odom_publish_frequency>10</odom_publish_frequency>
-            <odom_topic>/model/forklift/left_wheel/odometry</odom_topic>
-          </plugin>
-        <!--
-        <plugin
             filename="gz-sim-pose-publisher-system"
             name="gz::sim::systems::PosePublisher">
@@ -43,5 +29,4 @@
             <publish_nested_model_pose>true</publish_nested_model_pose>
         </plugin>
-        -->
       <plugin filename="gz-sim-joint-state-publisher-system" name="gz::sim::systems::JointStatePublisher">
           <topic>joint_states</topic>

File: src/test_bot_controller/urdf/robot_core.xacro (robot description, xacro)
@@ -27,4 +27,6 @@
         <child link="chassis"/>
         <origin xyz="0 0 0.125"/>
+        <axis xyz="0 0 1"/>
+        <limit effort="110" lower="0" upper="0.6" velocity="0.5"/>
     </joint>
     <link name="chassis">
@@ -48,5 +50,5 @@
     <link name="track_1">
         <visual>
-            <origin xyz="0 0 ${track_length/2 - base_height/2}" rpy="${pi/2} 0 ${pi/2}"/>
+            <origin xyz="0 0 0.09" rpy="${pi/2} 0 ${pi/2}"/>
             <geometry>
                 <box size="${track_width} ${track_length} ${track_depth}"/>
@@ -64,8 +66,10 @@
         </xacro:inertial_box>
     </link>
-    <joint name="track1_joint" type="fixed">
+    <joint name="track1_joint" type="prismatic">
         <parent link="chassis"/>
         <child link="track_1"/>
         <origin xyz="${base_width/2 + track_depth/2} ${base_width/2 - track_width} 0" rpy="0 0 0 " />
+        <axis xyz="0 0 1"/>
+        <limit effort="110" lower="0" upper="0.6" velocity="0.5"/>
     </joint>
     <link name="track_2">
@@ -87,25 +91,27 @@
         </xacro:inertial_box>
     </link>
-    <joint name="track2_joint" type="fixed">
+    <joint name="track2_joint" type="prismatic">
         <parent link="chassis"/>
         <child link="track_2"/>
         <origin xyz="${base_width/2 + track_depth/2} -${base_width/2 - track_width} 0" rpy="0 0 0" />
+        <axis xyz="0 0 1"/>
+        <limit effort="110" lower="0" upper="0.6" velocity="0.5"/>
     </joint>
     <link name="fork_plate">
         <visual>
-            <origin xyz="${track_depth/2} 0.1 0" rpy="0 ${pi/2} 0"/>
-            <geometry>
-                <box size="0.1 0.25 ${track_depth}"/>
-            </geometry>
-            <material name="blue"/>
-        </visual>
-        <collision>
-            <origin xyz="${track_depth/2} 0.1 0" rpy="0 ${pi/2} 0"/>
-            <geometry>
-                <box size="0.1 0.25 ${track_depth}"/>
-            </geometry>
-        </collision>
-        <xacro:inertial_box mass="10" x="0.1" y="0.25" z="${track_depth}">
-            <origin xyz="${track_depth/2} 0.1 0" rpy="0 ${pi/2} 0"/>
+            <origin xyz="0.0 0 0" rpy="0 0 0"/>
+            <geometry>
+                <box size="0.5 0.25 0.02"/>
+            </geometry>
+            <material name="blue"/>
+        </visual>
+        <collision>
+            <origin xyz="0 0 0" rpy="0 0 0"/>
+            <geometry>
+                <box size="0.5 0.25 0.2"/>
+            </geometry>
+        </collision>
+        <xacro:inertial_box mass="10" x="0" y="0" z="0">
+            <origin xyz="0.2 0.1 0" rpy="0 0 0"/>
         </xacro:inertial_box>
     </link>
@@ -114,5 +120,5 @@
         <child link="fork_plate"/>
         <!--Offset the joint position by the track depth amount-->
-        <origin xyz="${track_depth/2} 0 -0.025" rpy="0 0 0" />
+        <origin xyz="0.3 0 0" rpy="0 0 0" />
         <axis xyz="0 0 1"/>
         <limit effort="110" lower="0" upper="0.6" velocity="0.5"/>

Commit message: Add 3d model

File: src/test_bot_controller/urdf/robot.urdf.xacro (robot description, xacro)
@@ -1,4 +1,4 @@
 <?xml version="1.0"?>
-<robot xmlns:xacro="http://www.ros.org/wiki/xacro"  name="robot">
+<robot xmlns:xacro="http://www.ros.org/wiki/xacro"  name="forklift">
     <xacro:include filename="robot_core.xacro" />
     <gazebo>
@@ -21,4 +21,11 @@
             <odom_frame>base_link</odom_frame>
         </plugin>
+        <plugin filename="gz-sim-odometry-publisher-system" name="gz::sim::systems::OdometryPublisher" >
+            <odom_frame>world</odom_frame>
+            <robot_base_frame>forklift/left_wheel</robot_base_frame>
+            <odom_publish_frequency>10</odom_publish_frequency>
+            <odom_topic>/model/forklift/left_wheel/odometry</odom_topic>
+          </plugin>
+        <!--
         <plugin
             filename="gz-sim-pose-publisher-system"
@@ -29,4 +36,5 @@
             <publish_nested_model_pose>true</publish_nested_model_pose>
         </plugin>
+        -->
       <plugin filename="gz-sim-joint-state-publisher-system" name="gz::sim::systems::JointStatePublisher">
           <topic>joint_states</topic>

File: src/test_bot_controller/urdf/robot_core (Copy).xacro (robot description, xacro)
@@ -26,5 +26,5 @@
         <parent link="base_link"/>
         <child link="chassis"/>
-        <origin xyz="0 0 0.125"/>
+        <origin xyz="0 0 0.75"/>
         <axis xyz="0 0 1"/>
         <limit effort="110" lower="0" upper="0.6" velocity="0.5"/>
@@ -32,5 +32,5 @@
     <link name="chassis">
         <visual>
-            <origin xyz="0 0 0.02"/>
+            <origin xyz="0 0 0"/>
             <geometry>
                 <mesh filename="$(find test_bot_controller)/meshes/body.dae" scale="0.0027 0.0027 0.0027"/>
@@ -52,19 +52,17 @@
             <origin xyz="0 0 0" rpy="0 0 0"/>
             <geometry>
-                <!-- <box size="0.01 0.2 0.2"/> -->
                 <mesh filename="$(find test_bot_controller)/meshes/fork_plate.dae" scale="0.0027 0.0027 0.0027"/>
-            </geometry>
-        </visual>
-        <collision>
-            <origin xyz="0 0 0" rpy="0 0 0"/>
-            <geometry>
-                <box size="0.01 0.3 0.2"/>
-            </geometry>
-        </collision>
-        <inertial>
-            <mass value="75"/>
-            <origin xyz="0.005 0.15 0.1" rpy="0 0 0"/>
-            <inertia ixx="0.075" ixy="0" ixz="0" iyy="0.075" iyz="0" izz="0.0045"/>
-        </inertial>
+                <!-- <box size="0.1 0.25 0.02"/> -->
+            </geometry>
+        </visual>
+        <collision>
+            <origin xyz="0 0 0" rpy="0 0 0"/>
+            <geometry>
+                <mesh filename="$(find test_bot_controller)/meshes/fork_plate.dae" scale="0.0027 0.0027 0.0027"/>
+            </geometry>
+        </collision>
+        <xacro:inertial_box mass="10" x="0" y="0" z="0">
+            <origin xyz="0.2 0.1 0" rpy="0 0 0"/>
+        </xacro:inertial_box>
     </link>
     <joint name="fork_plate_joint" type="prismatic">
@@ -72,5 +70,5 @@
         <child link="fork_plate"/>
         <!--Offset the joint position by the track depth amount-->
-        <origin xyz="0.375 0 0" rpy="0 0 0"/>
+        <origin xyz="0.375 0 0" rpy="0 0 0" />
         <axis xyz="0 0 1"/>
         <limit effort="110" lower="0" upper="0.6" velocity="0.5"/>
@@ -78,44 +76,42 @@
     <link name="fork_1">
         <visual>
-            <origin xyz="0.15 0 0" rpy="0 0 0"/>
-            <geometry>
-                <box size="0.3 0.05 0.01"/>
-            </geometry>
-        </visual>
-        <collision>
-            <origin xyz="0.15 0 0" rpy="0 0 0"/>
-            <geometry>
-                <box size="0.3 0.05 0.01"/>
-            </geometry>
-        </collision>
-        <inertial>
-            <mass value="50"/>
-            <origin xyz="0.15 0 0" rpy="0 0 0"/>
-            <inertia ixx="0.00010417" ixy="0" ixz="0" iyy="0.06510417" iyz="0" izz="0.06510417"/>
-        </inertial>
+            <origin xyz="0 0 0" rpy="0 0 -${pi}"/>
+            <geometry>
+                <mesh filename="$(find test_bot_controller)/meshes/fork.dae" scale="0.0027 0.0027 0.0027"/>
+            </geometry>
+        </visual>
+        <collision>
+            <origin xyz="0 0 0" rpy="0 0 -${pi/2}"/>
+            <geometry>
+                <mesh filename="$(find test_bot_controller)/meshes/fork.dae" scale="0.0027 0.0027 0.0027"/>
+            </geometry>
+        </collision>
+        <xacro:inertial_box mass="10" x="0" y="0" z="0">
+            <origin xyz="0 0 0" rpy="0 0 -${pi/2}"/>
+        </xacro:inertial_box>
     </link>
     <joint name="fork_1_joint" type="fixed">
         <parent link="fork_plate"/>
         <child link="fork_1"/>
-        <origin xyz="0 -0.05 -0.01" rpy="0 0 0"/>
+        <!--Offset the joint position by the track depth amount-->
+        <origin xyz="-0.01 -0.075 -0.03" rpy="0 0 0" />
     </joint>
     <link name="fork_2">
         <visual>
-            <origin xyz="0.15 0 0" rpy="0 0 0"/>
-            <geometry>
-                <box size="0.3 0.05 0.01"/>
-            </geometry>
-        </visual>
-        <collision>
-            <origin xyz="0.15 0 0" rpy="0 0 0"/>
-            <geometry>
-                <box size="0.3 0.05 0.01"/>
-            </geometry>
-        </collision>
-        <inertial>
-            <mass value="50"/>
-            <origin xyz="0.15 0 0" rpy="0 0 0"/>
-            <inertia ixx="0.00010417" ixy="0" ixz="0" iyy="0.06510417" iyz="0" izz="0.06510417"/>
-        </inertial>
+            <origin xyz="0 0 0" rpy="0 0 -${pi/2}"/>
+            <geometry>
+                <box size="0.05 0.3 0.02"/>
+            </geometry>
+            <material name="white"/>
+        </visual>
+        <collision>
+            <origin xyz="0 0 0" rpy="0 0 -${pi/2}"/>
+            <geometry>
+                <box size="0.5 0.25 0.02"/>
+            </geometry>
+        </collision>
+        <xacro:inertial_box mass="10" x="0" y="0" z="0">
+            <origin xyz="0 0 0" rpy="0 0 -${pi/2}"/>
+        </xacro:inertial_box>
     </link>
     <joint name="fork_2_joint" type="fixed">
@@ -123,5 +119,7 @@
         <child link="fork_2"/>
         <!--Offset the joint position by the track depth amount-->
-        <origin xyz="0 0.05 -0.01" rpy="0 0 0"/>
+        <origin xyz="0.154 0.15 0" rpy="0 0 0" />
+        <axis xyz="0 0 1"/>
+        <limit effort="110" lower="0" upper="0.6" velocity="0.5"/>
     </joint>
     <!-- LEFT WHEEL LINK -->
@@ -129,18 +127,18 @@
         <parent link="chassis"/>
         <child link="left_wheel"/>
-        <origin xyz="0.23 0.13 -0.075" rpy="0 0 0" />
+        <origin xyz="0.225 0.125 -0.075" rpy="0 0 0" />
         <axis xyz="0 1 0"/>
     </joint>
     <link name="left_wheel">
-        <visual>
-            <origin xyz="0 0 0" rpy="0 0 0"/>
-            <geometry>
-                <mesh filename="$(find test_bot_controller)/meshes/front_wheel_right.dae" scale="0.002 0.002 0.002"/>
-            </geometry>
-        </visual>
-        <collision>
-            <origin xyz="0 0 0" rpy="-${pi/2} 0 0"/>
-            <geometry>
-                <cylinder radius="0.05" length="0.02"/>
+        <origin xyz="0 0 3" rpy="0 0 -${pi}"/>
+        <visual>
+            <geometry>
+                <cylinder radius="0.07" length="0.02"/>
+            </geometry>
+        </visual>
+        <collision>
+            <origin xyz="0 0 0" rpy="${pi/2} 0 0 "/>
+            <geometry>
+                <cylinder radius="0.07" length="0.02"/>
             </geometry>
         </collision>
@@ -152,19 +150,17 @@
         <parent link="chassis"/>
         <child link="left_wheel_back"/>
-        <origin xyz="-0.10 0.155 -0.075" rpy="0 0 0" />
+        <origin xyz="-0.2 0.125 -0.075" rpy="0 0 0" />
         <axis xyz="0 1 0"/>
     </joint>
     <link name="left_wheel_back">
         <visual>
-            <origin xyz="0 0 0" rpy="0 0 0"/>
-            <geometry>
-                <mesh filename="$(find test_bot_controller)/meshes/back_wheel_left.dae" scale="0.002 0.002 0.002"/>
-                <!-- <cylinder radius="0.05" length="0.02"/> -->
-            </geometry>
-        </visual>
-        <collision>
-            <origin xyz="0 0 0" rpy="-${pi/2} 0 0"/>
-            <geometry>
-                <cylinder radius="0.05" length="0.02"/>
+            <geometry>
+                <cylinder radius="0.07" length="0.02"/>
+            </geometry>
+        </visual>
+        <collision>
+            <origin xyz="0 0 0" rpy="${pi/2} 0 0 "/>
+            <geometry>
+                <cylinder radius="0.07" length="0.02"/>
             </geometry>
         </collision>
@@ -177,22 +173,21 @@
         <parent link="chassis"/>
         <child link="right_wheel"/>
-        <origin xyz="0.23 -0.13 -0.075" rpy="0 0 0" />
+        <origin xyz="0.225 -0.125 -0.075" rpy="0 0 0" />
         <axis xyz="0 1 0"/>
     </joint>
     <link name="right_wheel">
         <visual>
-            <origin xyz="0 0 0" rpy="0 0 0"/>
-            <geometry>
-                <mesh filename="$(find test_bot_controller)/meshes/front_wheel_right.dae" scale="0.002 0.002 0.002"/>
-            </geometry>
-        </visual>
-        <collision>
-            <origin xyz="0 0 0" rpy="-${pi/2} 0 0"/>
-            <geometry>
-                <cylinder radius="0.05" length="0.02"/>
-            </geometry>
-        </collision>
-        <xacro:inertial_cylinder mass="0.1" length="0.02" radius="0.05">
-            <origin xyz="0 0 0" rpy="-${pi/2} 0 0"/>
+            <geometry>
+                <cylinder radius="0.07" length="0.02"/>
+            </geometry>
+        </visual>
+        <collision>
+            <origin xyz="0 0 0" rpy="${pi/2} 0 0 "/>
+            <geometry>
+                <cylinder radius="0.07" length="0.02"/>
+            </geometry>
+        </collision>
+        <xacro:inertial_cylinder mass="0.1" length="0.02" radius="0.05">
+            <origin xyz="0 0 0" rpy="0 0 0"/>
         </xacro:inertial_cylinder>
     </link>
@@ -200,17 +195,17 @@
         <parent link="chassis"/>
         <child link="right_wheel_back"/>
-        <origin xyz="-0.10 -0.155 -0.075" rpy="${pi/2} 0 0" />
-        <axis xyz="0 0 -1"/>
+        <origin xyz="-0.2 -0.125 -0.075" rpy="0 0 0" />
+        <axis xyz="0 1 0"/>
     </joint>
     <link name="right_wheel_back">
         <visual>
             <geometry>
-                <cylinder radius="0.05" length="0.02"/>
-            </geometry>
-            <material name="blue"/>
-        </visual>
-        <collision>
-            <geometry>
-                <cylinder radius="0.05" length="0.02"/>
+                <cylinder radius="0.07" length="0.02"/>
+            </geometry>
+        </visual>
+        <collision>
+            <origin xyz="0 0 0" rpy="${pi/2} 0 0 "/>
+            <geometry>
+                <cylinder radius="0.07" length="0.02"/>
             </geometry>
         </collision>
