Commit message: Implement pickup

File: src/test_bot_controller/urdf/robot.urdf.xacro (robot description, xacro)
@@ -11,5 +11,5 @@
             <right_joint>right_wheel_back_joint</right_joint>
             <wheel_separation>0.3</wheel_separation>
-            <wheel_radius>0.05</wheel_radius>
+            <wheel_radius>0.07</wheel_radius>
             <odom_publish_frequency>1</odom_publish_frequency>
             <topic>cmd_vel</topic>

File: src/test_bot_controller/urdf/robot_core.xacro (robot description, xacro)
@@ -32,5 +32,5 @@
     <link name="chassis">
         <visual>
-            <origin xyz="0 0 0.02"/>
+            <origin xyz="0 0 0.05"/>
             <geometry>
                 <mesh filename="$(find test_bot_controller)/meshes/body.dae" scale="0.0027 0.0027 0.0027"/>
@@ -142,5 +142,5 @@
             <origin xyz="0 0 0" rpy="-${pi/2} 0 0"/>
             <geometry>
-                <cylinder radius="0.05" length="0.02"/>
+                <cylinder radius="0.07" length="0.02"/>
             </geometry>
         </collision>
@@ -152,12 +152,12 @@
         <parent link="chassis"/>
         <child link="left_wheel_back"/>
-        <origin xyz="-0.10 0.155 -0.075" rpy="0 0 0" />
+        <origin xyz="-0.2 0.13 -0.075" rpy="0 0 0" />
         <axis xyz="0 1 0"/>
     </joint>
     <link name="left_wheel_back">
         <visual>
-            <origin xyz="0 0 0" rpy="0 0 0"/>
-            <geometry>
-                <mesh filename="$(find test_bot_controller)/meshes/back_wheel_left.dae" scale="0.002 0.002 0.002"/>
+            <origin xyz="0 0 0" rpy="0 0 ${pi}"/>
+            <geometry>
+                <mesh filename="$(find test_bot_controller)/meshes/front_wheel_right.dae" scale="0.002 0.002 0.002"/>
                 <!-- <cylinder radius="0.05" length="0.02"/> -->
             </geometry>
@@ -166,5 +166,5 @@
             <origin xyz="0 0 0" rpy="-${pi/2} 0 0"/>
             <geometry>
-                <cylinder radius="0.05" length="0.02"/>
+                <cylinder radius="0.07" length="0.02"/>
             </geometry>
         </collision>
@@ -190,5 +190,5 @@
             <origin xyz="0 0 0" rpy="-${pi/2} 0 0"/>
             <geometry>
-                <cylinder radius="0.05" length="0.02"/>
+                <cylinder radius="0.07" length="0.02"/>
             </geometry>
         </collision>
@@ -200,21 +200,21 @@
         <parent link="chassis"/>
         <child link="right_wheel_back"/>
-        <origin xyz="-0.10 -0.155 -0.075" rpy="${pi/2} 0 0" />
-        <axis xyz="0 0 -1"/>
+        <origin xyz="-0.2 -0.13 -0.075" rpy="0 0 0" />
+        <axis xyz="0 1 0"/>
     </joint>
     <link name="right_wheel_back">
         <visual>
             <geometry>
-                <cylinder radius="0.05" length="0.02"/>
-            </geometry>
-            <material name="blue"/>
-        </visual>
-        <collision>
-            <geometry>
-                <cylinder radius="0.05" length="0.02"/>
-            </geometry>
-        </collision>
-        <xacro:inertial_cylinder mass="0.1" length="0.02" radius="0.05">
-            <origin xyz="0 0 0" rpy="0 0 0"/>
+                <mesh filename="$(find test_bot_controller)/meshes/front_wheel_right.dae" scale="0.002 0.002 0.002"/>
+            </geometry>
+        </visual>
+        <collision>
+            <origin xyz="0 0 0" rpy="-${pi/2} 0 0"/>
+            <geometry>
+                <cylinder radius="0.07" length="0.02"/>
+            </geometry>
+        </collision>
+        <xacro:inertial_cylinder mass="0.1" length="0.02" radius="0.05">
+            <origin xyz="0 0 0" rpy="-${pi/2} 0 0"/>
         </xacro:inertial_cylinder>
     </link>

Commit message: Implement drop functionality

File: src/test_bot_controller/urdf/robot.urdf.xacro (robot description, xacro)
@@ -21,11 +21,4 @@
             <odom_frame>base_link</odom_frame>
         </plugin>
-        <plugin filename="gz-sim-odometry-publisher-system" name="gz::sim::systems::OdometryPublisher" >
-            <odom_frame>world</odom_frame>
-            <robot_base_frame>forklift/left_wheel</robot_base_frame>
-            <odom_publish_frequency>10</odom_publish_frequency>
-            <odom_topic>/model/forklift/left_wheel/odometry</odom_topic>
-          </plugin>
-        <!--
         <plugin
             filename="gz-sim-pose-publisher-system"
@@ -36,5 +29,4 @@
             <publish_nested_model_pose>true</publish_nested_model_pose>
         </plugin>
-        -->
       <plugin filename="gz-sim-joint-state-publisher-system" name="gz::sim::systems::JointStatePublisher">
           <topic>joint_states</topic>

File: src/test_bot_controller/urdf/robot_core.xacro (robot description, xacro)
@@ -20,15 +20,13 @@
     <xacro:property name="base_height" value="0.15"/>
     <xacro:property name="base_width" value="0.3"/>
+    <link name="base_footprint">
+    </link>
+    <!-- base_link LINK -->
+    <joint name="base_link_joint" type="fixed">
+        <parent link="base_footprint"/>
+        <child link="base_link"/>
+        <origin xyz="0 0 0.125"/>
+    </joint>
     <link name="base_link">
-    </link>
-    <!-- CHASSIS LINK -->
-    <joint name="chassis_joint" type="fixed">
-        <parent link="base_link"/>
-        <child link="chassis"/>
-        <origin xyz="0 0 0.125"/>
-        <axis xyz="0 0 1"/>
-        <limit effort="110" lower="0" upper="0.6" velocity="0.5"/>
-    </joint>
-    <link name="chassis">
         <visual>
             <origin xyz="0 0 0.05"/>
@@ -69,5 +67,5 @@
     </link>
     <joint name="fork_plate_joint" type="prismatic">
-        <parent link="chassis"/>
+        <parent link="base_link"/>
         <child link="fork_plate"/>
         <!--Offset the joint position by the track depth amount-->
@@ -127,5 +125,5 @@
     <!-- LEFT WHEEL LINK -->
     <joint name="left_wheel_joint" type="continuous">
-        <parent link="chassis"/>
+        <parent link="base_link"/>
         <child link="left_wheel"/>
         <origin xyz="0.23 0.13 -0.075" rpy="0 0 0" />
@@ -150,5 +148,5 @@
     </link>
     <joint name="left_wheel_back_joint" type="continuous">
-        <parent link="chassis"/>
+        <parent link="base_link"/>
         <child link="left_wheel_back"/>
         <origin xyz="-0.2 0.13 -0.075" rpy="0 0 0" />
@@ -175,5 +173,5 @@
     <!-- RIGHT WHEEL LINK -->
     <joint name="right_wheel_joint" type="continuous">
-        <parent link="chassis"/>
+        <parent link="base_link"/>
         <child link="right_wheel"/>
         <origin xyz="0.23 -0.13 -0.075" rpy="0 0 0" />
@@ -198,5 +196,5 @@
     </link>
     <joint name="right_wheel_back_joint" type="continuous">
-        <parent link="chassis"/>
+        <parent link="base_link"/>
         <child link="right_wheel_back"/>
         <origin xyz="-0.2 -0.13 -0.075" rpy="0 0 0" />
