Commit message: Rename package

File: src/forklift_controller/urdf/robot_core (Copy).xacro (robot description, xacro)
@@ -34,5 +34,5 @@
             <origin xyz="0 0 0"/>
             <geometry>
-                <mesh filename="$(find test_bot_controller)/meshes/body.dae" scale="0.0027 0.0027 0.0027"/>
+                <mesh filename="$(find forklift_controller)/meshes/body.dae" scale="0.0027 0.0027 0.0027"/>
                 <!-- <box size="0.3 ${base_width} ${base_height}"/> -->
             </geometry>
@@ -52,5 +52,5 @@
             <origin xyz="0 0 0" rpy="0 0 0"/>
             <geometry>
-                <mesh filename="$(find test_bot_controller)/meshes/fork_plate.dae" scale="0.0027 0.0027 0.0027"/>
+                <mesh filename="$(find forklift_controller)/meshes/fork_plate.dae" scale="0.0027 0.0027 0.0027"/>
                 <!-- <box size="0.1 0.25 0.02"/> -->
             </geometry>
@@ -59,5 +59,5 @@
             <origin xyz="0 0 0" rpy="0 0 0"/>
             <geometry>
-                <mesh filename="$(find test_bot_controller)/meshes/fork_plate.dae" scale="0.0027 0.0027 0.0027"/>
+                <mesh filename="$(find forklift_controller)/meshes/fork_plate.dae" scale="0.0027 0.0027 0.0027"/>
             </geometry>
         </collision>
@@ -78,11 +78,11 @@
             <origin xyz="0 0 0" rpy="0 0 -${pi}"/>
             <geometry>
-                <mesh filename="$(find test_bot_controller)/meshes/fork.dae" scale="0.0027 0.0027 0.0027"/>
-            </geometry>
-        </visual>
-        <collision>
-            <origin xyz="0 0 0" rpy="0 0 -${pi/2}"/>
-            <geometry>
-                <mesh filename="$(find test_bot_controller)/meshes/fork.dae" scale="0.0027 0.0027 0.0027"/>
+                <mesh filename="$(find forklift_controller)/meshes/fork.dae" scale="0.0027 0.0027 0.0027"/>
+            </geometry>
+        </visual>
+        <collision>
+            <origin xyz="0 0 0" rpy="0 0 -${pi/2}"/>
+            <geometry>
+                <mesh filename="$(find forklift_controller)/meshes/fork.dae" scale="0.0027 0.0027 0.0027"/>
             </geometry>
         </collision>

File: src/forklift_controller/urdf/robot_core.xacro (robot description, xacro)
@@ -32,5 +32,5 @@
             <origin xyz="0 0 0.05"/>
             <geometry>
-                <mesh filename="$(find test_bot_controller)/meshes/body.dae" scale="0.0027 0.0027 0.0027"/>
+                <mesh filename="$(find forklift_controller)/meshes/body.dae" scale="0.0027 0.0027 0.0027"/>
                 <!-- <box size="0.3 ${base_width} ${base_height}"/> -->
             </geometry>
@@ -51,5 +51,5 @@
             <geometry>
                 <!-- <box size="0.01 0.2 0.2"/> -->
-                <mesh filename="$(find test_bot_controller)/meshes/fork_plate.dae" scale="0.0027 0.0027 0.0027"/>
+                <mesh filename="$(find forklift_controller)/meshes/fork_plate.dae" scale="0.0027 0.0027 0.0027"/>
             </geometry>
         </visual>
@@ -134,5 +134,5 @@
             <origin xyz="0 0 0" rpy="0 0 0"/>
             <geometry>
-                <mesh filename="$(find test_bot_controller)/meshes/front_wheel_right.dae" scale="0.002 0.002 0.002"/>
+                <mesh filename="$(find forklift_controller)/meshes/front_wheel_right.dae" scale="0.002 0.002 0.002"/>
             </geometry>
         </visual>
@@ -157,5 +157,5 @@
             <origin xyz="0 0 0" rpy="0 0 ${pi}"/>
             <geometry>
-                <mesh filename="$(find test_bot_controller)/meshes/front_wheel_right.dae" scale="0.002 0.002 0.002"/>
+                <mesh filename="$(find forklift_controller)/meshes/front_wheel_right.dae" scale="0.002 0.002 0.002"/>
                 <!-- <cylinder radius="0.05" length="0.02"/> -->
             </geometry>
@@ -182,5 +182,5 @@
             <origin xyz="0 0 0" rpy="0 0 0"/>
             <geometry>
-                <mesh filename="$(find test_bot_controller)/meshes/front_wheel_right.dae" scale="0.002 0.002 0.002"/>
+                <mesh filename="$(find forklift_controller)/meshes/front_wheel_right.dae" scale="0.002 0.002 0.002"/>
             </geometry>
         </visual>
@@ -204,5 +204,5 @@
         <visual>
             <geometry>
-                <mesh filename="$(find test_bot_controller)/meshes/front_wheel_right.dae" scale="0.002 0.002 0.002"/>
+                <mesh filename="$(find forklift_controller)/meshes/front_wheel_right.dae" scale="0.002 0.002 0.002"/>
             </geometry>
         </visual>
