Commit message: Update joint state plugin

File: src/forklift_controller/urdf/fork.xacro (robot description, xacro)
@@ -1,6 +1,6 @@
 <?xml version="1.0"?>
-<robot xmlns:xacro="http://www.ros.org/wiki/xacro" >
-    <xacro:macro name="fork" params="id mass scale fork_attach_offsets">
-    <xacro:include filename="inertial_macros.xacro"/>
+<robot xmlns:xacro="http://www.ros.org/wiki/xacro">
+  <xacro:macro name="fork" params="id mass scale fork_attach_offsets">
+    <xacro:include filename="inertial_macros.xacro" />
     <!--
     Dimensions are defined when viewing link from the front:
@@ -9,64 +9,67 @@
       width is sideways (left/right)
     -->
-    <xacro:property name="fork_attach_height" value="0.15"/>
-    <xacro:property name="fork_attach_length" value="0.01"/>
-    <xacro:property name="fork_attach_width" value="0.025"/>
-    <xacro:property name="fork_visual_offset" value="0.04"/>
+    <xacro:property name="fork_attach_height" value="0.15" />
+    <xacro:property name="fork_attach_length" value="0.01" />
+    <xacro:property name="fork_attach_width" value="0.025" />
+    <xacro:property name="fork_visual_offset" value="0.04" />
+    <xacro:property name="fork_height" value="0.005" />
+    <xacro:property name="fork_length" value="0.2" />
+    <xacro:property name="fork_width" value="0.025" />
     <link name="fork_${id}_attach">
-        <visual>
-          <origin xyz="0 0 -${fork_visual_offset}" rpy="0 -${pi/2} 0"/>
+      <visual>
+        <origin xyz="0 0 -${fork_visual_offset}" rpy="0 -${pi/2} 0" />
+        <geometry>
+          <box size="${fork_attach_height} ${fork_attach_width} ${fork_attach_length}" />
+        </geometry>
+        <material name="darkgray" />
+      </visual>
+      <collision>
+        <origin xyz="0 0 -${fork_visual_offset}" rpy="0 -${pi/2} 0" />
+        <geometry>
+          <box size="${fork_attach_height} ${fork_attach_width} ${fork_attach_length}" />
+        </geometry>
+      </collision>
+      <xacro:inertial_box mass="${mass / 2}" x="${fork_attach_height}" y="${fork_attach_width}"
+        z="${fork_attach_length}">
+        <origin xyz="0 0 0" rpy="0 0 0" />
+      </xacro:inertial_box>
+    </link>
+    <link name="fork_${id}">
+      <visual>
+        <origin xyz="${fork_length/2} 0 0" rpy="0 0 0" />
+        <geometry>
+          <box size="${fork_length} ${fork_width} ${fork_height}" />
+        </geometry>
+        <material name="darkgray" />
+      </visual>
+      <collision>
+        <origin xyz="${fork_length/2} 0 0" rpy="0 0 0" />
+        <geometry>
+          <box size="${fork_length} ${fork_width} ${fork_height}" />
+        </geometry>
+        <!--
             <geometry>
-              <box size="${fork_attach_height} ${fork_attach_width} ${fork_attach_length}"/>
-            </geometry>
-            <material name="darkgray" />
-        </visual>
-        <collision>
-          <origin xyz="0 0 -${fork_visual_offset}" rpy="0 -${pi/2} 0"/>
-          <geometry>
-            <box size="${fork_attach_height} ${fork_attach_width} ${fork_attach_length}"/>
-          </geometry>
-        </collision>
-          <xacro:inertial_box mass="${mass / 2}" x="${fork_attach_height}" y="${fork_attach_width}" z="${fork_attach_length}">
-            <origin xyz="0 0 0" rpy="0 0 0"/>
-        </xacro:inertial_box>
-      </link>
-    <xacro:property name="fork_height" value="0.005"/>
-    <xacro:property name="fork_length" value="0.2"/>
-    <xacro:property name="fork_width" value="0.025"/>
-    <link name="fork_${id}">
-        <visual>
-          <origin xyz="${fork_length/2} 0 0" rpy="0 0 0"/>
-          <geometry>
-            <box size="${fork_length} ${fork_width} ${fork_height}"/>
-          </geometry>
-            <material name="darkgray" />
-        </visual>
-        <collision>
-          <origin xyz="${fork_length/2} 0 0" rpy="0 0 0"/>
-          <!-- <origin xyz="0 0 0"  rpy="0 0 -${pi}"/> -->
-            <geometry>
-                <box size="${fork_length} ${fork_width} ${fork_height}"/>
-            </geometry>
-            <!--
-            <geometry>
-                <mesh filename="$(find forklift_controller)/models/forklift/meshes/fork.dae" scale="0.0027 0.0027 0.0027"/>
+                <mesh filename="$(find forklift_controller)/models/forklift/meshes/fork.dae" scale="0.0027 0.0027
+        0.0027"/>
             </geometry>
             -->
-        </collision>
-          <xacro:inertial_box mass="${mass / 2}" x="${fork_length}" y="${fork_width}" z="${fork_height}">
-            <origin xyz="0 0 0" rpy="0 0 0"/>
-        </xacro:inertial_box>
+      </collision>
+      <xacro:inertial_box mass="${mass / 2}" x="${fork_length}" y="${fork_width}" z="${fork_height}">
+        <origin xyz="0 0 0" rpy="0 0 0" />
+      </xacro:inertial_box>
     </link>
     <joint name="fork_attach_${id}_joint" type="fixed">
-        <parent link="fork_plate"/>
-        <child link="fork_${id}_attach"/>
-        <origin xyz="${fork_attach_offsets}" rpy="0 0 0"/>
+      <parent link="fork_plate" />
+      <child link="fork_${id}_attach" />
+      <origin xyz="${fork_attach_offsets}" rpy="0 0 0" />
     </joint>
-      <joint name="fork_${id}_joint" type="fixed">
-          <parent link="fork_${id}_attach"/>
-          <child link="fork_${id}"/>
-          <origin xyz="${0.01/2} 0 -${fork_attach_height - fork_visual_offset + fork_height/2}" rpy="0 0 0"/>
-      </joint>
+    <joint name="fork_${id}_joint" type="fixed">
+      <parent link="fork_${id}_attach" />
+      <child link="fork_${id}" />
+      <origin xyz="${0.01/2} 0 -${fork_attach_height - fork_visual_offset + fork_height/2}"
+        rpy="0 0 0" />
+    </joint>
     <!-- https://osrf-migration.github.io/sdformat-gh-pages/#!/osrf/sdformat/issues/131/page/1-->
+    <!--
     <gazebo reference="fork_{id}_joint">
         <disableFixedJointLumping>true</disableFixedJointLumping>
@@ -75,4 +78,5 @@
         <disableFixedJointLumping>true</disableFixedJointLumping>
     </gazebo>
-    </xacro:macro>
+    -->
+  </xacro:macro>
 </robot>

File: src/forklift_controller/urdf/robot.urdf.xacro (robot description, xacro)
@@ -1,38 +1,32 @@
 <?xml version="1.0"?>
-<robot xmlns:xacro="http://www.ros.org/wiki/xacro"  name="forklift">
-    <xacro:arg name="namespace" default=""/>
-    <xacro:include filename="robot_core.xacro" />
-    <gazebo>
-        <plugin
-        filename="gz-sim-diff-drive-system"
-        name="gz::sim::systems::DiffDrive">
-            <left_joint>left_wheel_joint</left_joint>
-            <left_joint>left_wheel_back_joint</left_joint>
-            <right_joint>right_wheel_joint</right_joint>
-            <right_joint>right_wheel_back_joint</right_joint>
-            <wheel_separation>0.26</wheel_separation>
-            <wheel_radius>0.07</wheel_radius>
-            <odom_publish_frequency>30</odom_publish_frequency>
-            <odom_topic>$(arg namespace)/odom</odom_topic>
-            <frame_id>odom</frame_id>
-            <tf_topic>$(arg namespace)/tf</tf_topic>
-            <topic>$(arg namespace)/cmd_vel</topic>
-            <child_frame_id>base_link</child_frame_id>
-            <max_linear_acceleration>10</max_linear_acceleration>
-            <min_linear_acceleration>-10</min_linear_acceleration>
-            <max_angular_acceleration>20</max_angular_acceleration>
-            <min_angular_acceleration>-20</min_angular_acceleration>
-            <max_linear_velocity>0.5</max_linear_velocity>
-            <min_linear_velocity>-0.5</min_linear_velocity>
-            <max_angular_velocity>10</max_angular_velocity>
-            <min_angular_velocity>-10</min_angular_velocity>
-        </plugin>
-        <!--
-        <plugin
-        filename="gz-sim-odometry-publisher-system"
-        name="gz::sim::systems::OdometryPublisher">
-            <odom_frame>base_link</odom_frame>
-            <odom_topic>$(arg namespace)/odometry</odom_topic>
-        </plugin>
+<robot xmlns:xacro="http://www.ros.org/wiki/xacro" name="forklift">
+  <xacro:arg name="namespace" default="" />
+  <xacro:include filename="robot_core.xacro" />
+  <gazebo>
+    <plugin
+      filename="gz-sim-diff-drive-system"
+      name="gz::sim::systems::DiffDrive">
+      <left_joint>left_wheel_joint</left_joint>
+      <left_joint>left_wheel_back_joint</left_joint>
+      <right_joint>right_wheel_joint</right_joint>
+      <right_joint>right_wheel_back_joint</right_joint>
+      <wheel_separation>0.26</wheel_separation>
+      <wheel_radius>0.07</wheel_radius>
+      <odom_publish_frequency>30</odom_publish_frequency>
+      <odom_topic>$(arg namespace)/odom</odom_topic>
+      <frame_id>odom</frame_id>
+      <tf_topic>$(arg namespace)/tf</tf_topic>
+      <topic>$(arg namespace)/cmd_vel</topic>
+      <child_frame_id>base_link</child_frame_id>
+      <max_linear_acceleration>10</max_linear_acceleration>
+      <min_linear_acceleration>-10</min_linear_acceleration>
+      <max_angular_acceleration>20</max_angular_acceleration>
+      <min_angular_acceleration>-20</min_angular_acceleration>
+      <max_linear_velocity>0.5</max_linear_velocity>
+      <min_linear_velocity>-0.5</min_linear_velocity>
+      <max_angular_velocity>10</max_angular_velocity>
+      <min_angular_velocity>-10</min_angular_velocity>
+    </plugin>
+    <!--
         <plugin
             filename="gz-sim-pose-publisher-system"
@@ -44,13 +38,19 @@
         </plugin>
         -->
-      <plugin filename="gz-sim-joint-state-publisher-system" name="gz::sim::systems::JointStatePublisher">
-        <joint_name>left_wheel_joint</joint_name>
-        <joint_name>right_wheel_joint</joint_name>
-        <joint_name>left_wheel_back_joint</joint_name>
-        <joint_name>right_wheel_back_joint</joint_name>
-        <topic>$(arg namespace)/joint_states</topic>
-      </plugin>
-      <!--
-      <plugin filename="gz-sim-joint-position-controller-system" name="gz::sim::systems::JointPositionController">
+    <plugin filename="gz-sim-joint-state-publisher-system"
+      name="gz::sim::systems::JointStatePublisher">
+      <joint_name>left_wheel_joint</joint_name>
+      <joint_name>right_wheel_joint</joint_name>
+      <joint_name>left_wheel_back_joint</joint_name>
+      <joint_name>right_wheel_back_joint</joint_name>
+      <joint_name>fork_attach_1_joint</joint_name>
+      <joint_name>fork_attach_2_joint</joint_name>
+      <joint_name>fork_1_joint</joint_name>
+      <joint_name>fork_2_joint</joint_name>
+      <topic>$(arg namespace)/joint_states</topic>
+    </plugin>
+    <!--
+      <plugin filename="gz-sim-joint-position-controller-system"
+    name="gz::sim::systems::JointPositionController">
         <joint_name>fork_plate_joint</joint_name>
         <topic>fork_control</topic>
@@ -58,4 +58,4 @@
       </plugin>
       -->
-    </gazebo>
+  </gazebo>
 </robot>
