Commit message: Finish appropriate scaling with forklift

File: src/forklift_controller/urdf/fork.xacro (robot description, xacro)
@@ -9,14 +9,14 @@
       width is sideways (left/right)
     -->
-    <xacro:property name="fork_attach_height" value="0.15" />
-    <xacro:property name="fork_attach_length" value="0.01" />
+    <xacro:property name="fork_attach_height" value="0.5" />
+    <xacro:property name="fork_attach_length" value="0.1" />
     <xacro:property name="fork_attach_width" value="0.025" />
     <xacro:property name="fork_visual_offset" value="0.04" />
-    <xacro:property name="fork_height" value="0.005" />
-    <xacro:property name="fork_length" value="0.2" />
-    <xacro:property name="fork_width" value="0.025" />
+    <xacro:property name="fork_height" value="0.04" />
+    <xacro:property name="fork_length" value="1.0" />
+    <xacro:property name="fork_width" value="0.1" />
     <link name="fork_${id}_attach">
       <visual>
-        <origin xyz="0 0 -${fork_visual_offset}" rpy="0 -${pi/2} 0" />
+        <origin xyz="0 0 0" rpy="${pi/2} ${pi/2} 0" />
         <geometry>
           <box size="${fork_attach_height} ${fork_attach_width} ${fork_attach_length}" />
@@ -25,5 +25,5 @@
       </visual>
       <collision>
-        <origin xyz="0 0 -${fork_visual_offset}" rpy="0 -${pi/2} 0" />
+        <origin xyz="0 0 0" rpy="${pi/2} ${pi/2} 0" />
         <geometry>
           <box size="${fork_attach_height} ${fork_attach_width} ${fork_attach_length}" />
@@ -37,5 +37,5 @@
     <link name="fork_${id}">
       <visual>
-        <origin xyz="${fork_length/2} 0 0" rpy="0 0 0" />
+        <origin xyz="0 0 0" rpy="0 0 0" />
         <geometry>
           <box size="${fork_length} ${fork_width} ${fork_height}" />
@@ -44,14 +44,8 @@
       </visual>
       <collision>
-        <origin xyz="${fork_length/2} 0 0" rpy="0 0 0" />
+        <origin xyz="0 0 0" rpy="0 0 0" />
         <geometry>
           <box size="${fork_length} ${fork_width} ${fork_height}" />
         </geometry>
-        <!--
-            <geometry>
-                <mesh filename="$(find forklift_controller)/models/forklift/meshes/fork.dae" scale="0.0027 0.0027
-        0.0027"/>
-            </geometry>
-            -->
       </collision>
       <xacro:inertial_box mass="${mass / 2}" x="${fork_length}" y="${fork_width}" z="${fork_height}">
@@ -67,6 +61,5 @@
       <parent link="fork_${id}_attach" />
       <child link="fork_${id}" />
-      <origin xyz="${0.01/2} 0 -${fork_attach_height - fork_visual_offset + fork_height/2}"
-        rpy="0 0 0" />
+      <origin xyz="${fork_length/2} 0 -${fork_attach_height/2-fork_height/2}" rpy="0 0 0" />
     </joint>
     <!-- https://osrf-migration.github.io/sdformat-gh-pages/#!/osrf/sdformat/issues/131/page/1-->

File: src/forklift_controller/urdf/robot.urdf.xacro (robot description, xacro)
@@ -11,5 +11,5 @@
       <right_joint>right_wheel_joint</right_joint>
       <right_joint>right_wheel_back_joint</right_joint>
-      <wheel_separation>0.26</wheel_separation>
+      <wheel_separation>0.895</wheel_separation>
       <wheel_radius>0.07</wheel_radius>
       <odom_publish_frequency>30</odom_publish_frequency>

File: src/forklift_controller/urdf/robot_core.xacro (robot description, xacro)
@@ -3,4 +3,5 @@
   <xacro:include filename="inertial_macros.xacro" />
   <xacro:include filename="fork.xacro" />
+  <xacro:include filename="wheel.xacro"/>
   <material name="white">
     <color rgba="1 1 1 1" />
@@ -8,12 +9,7 @@
   <!-- BASE LINK -->
   <xacro:property name="scaler" value="1.0" />
-  <xacro:property name="track_length" value="0.3" />
-  <xacro:property name="track_depth" value="0.02" /> <!--This
-  is actually the depth of the track when in up position-->
-  <xacro:property name="track_width" value="0.05" /> <!--This
-  is actually the depth of the track when in up position-->
-  <xacro:property name="base_height" value="0.52" />
-  <xacro:property name="base_width" value="0.3" />
-  <xacro:property name="base_length" value="0.66" />
+  <xacro:property name="base_height" value="2" />
+  <xacro:property name="base_width" value="0.895" />
+  <xacro:property name="base_length" value="2.29" />
   <material name="darkgray">
     <color rgba="0.01 0.01 0.01 1" />
@@ -29,5 +25,5 @@
       <origin rpy="0 0 0" xyz="0 0 0" />
       <geometry>
-        <box size="${scaler*0.001} ${scaler*0.001} ${scaler*0.001}" />
+        <box size="0.001 0.001 0.001" />
       </geometry>
     </visual>
@@ -36,5 +32,6 @@
     <parent link="base_link" />
     <child link="base_footprint" />
-    <origin xyz="${scaler*0} ${scaler*0} ${scaler*-0.15}" rpy="0 0 0" />
+    <!--Set the base_footprint down to wheel axis level + half the wheel radius to be exactly at the bottom-->
+    <origin xyz="0 0 -${0.35+0.25}" rpy="0 0 0" />
   </joint>
   <link name="base_link">
@@ -42,12 +39,10 @@
       <origin xyz="0 0 0" />
       <geometry>
-        <mesh filename="package://forklift_controller/models/forklift/meshes/body.dae"
-          scale="0.0027 0.0027 0.0027" />
+        <mesh filename="package://forklift_controller/models/forklift/meshes/body_correct_scale.dae"/>
       </geometry>
     </visual>
     <collision>
       <geometry>
-        <mesh filename="package://forklift_controller/models/forklift/meshes/body.dae"
-          scale="${scaler*0.0027} ${scaler*0.0027} ${scaler*0.0027}" />
+        <mesh filename="package://forklift_controller/models/forklift/meshes/body_correct_scale.dae"/>
       </geometry>
     </collision>
@@ -56,10 +51,14 @@
     </xacro:inertial_box>
   </link>
+  <xacro:property name="plate_width" value="0.885"/>
+  <xacro:property name="plate_height" value="1.290"/>
+  <xacro:property name="plate_length" value="0.1"/>
   <link name="fork_plate">
     <visual>
       <origin xyz="0 0 0" rpy="0 0 0" />
       <geometry>
-        <mesh filename="package://forklift_controller/models/forklift/meshes/fork_plate.dae"
-          scale="0.0027 0.0027 0.0027" />
+        <mesh filename="package://forklift_controller/models/forklift/meshes/fork_plate_correct_scale.dae"
+        scale="1 1 0.77"
+        />
       </geometry>
     </visual>
@@ -67,8 +66,8 @@
       <origin xyz="0 0 0" rpy="0 0 0" />
       <geometry>
-        <box size="0.01 0.3 0.2" />
+        <box size="${plate_length} ${plate_width} ${plate_height}" />
       </geometry>
     </collision>
-    <xacro:inertial_box mass="50" x="0.01" y="0.3" z="0.2">
+    <xacro:inertial_box mass="50" x="${plate_length}" y="${plate_width}" z="${plate_height}">
       <origin xyz="0 0 0" rpy="0 0 0" />
     </xacro:inertial_box>
@@ -77,64 +76,14 @@
     <parent link="base_link" />
     <child link="fork_plate" />
-    <origin xyz="0.375 0 -0.02" rpy="0 0 0" />
+    <origin xyz="1.25 0 0.3" rpy="0 0 0" />
     <axis xyz="0 0 1" />
-    <limit effort="110" lower="0" upper="0.6" velocity="0.5" />
+    <limit effort="110" lower="-0.15" upper="0.6" velocity="0.5" />
   </joint>
-  <xacro:fork id="1" mass="15" scale="1" fork_attach_offsets="0.01 -0.05 -0.03"></xacro:fork>
-  <xacro:fork id="2" mass="15" scale="1" fork_attach_offsets="0.01 0.05 -0.03"></xacro:fork>
-  <!-- LEFT WHEEL LINK -->
-  <joint name="left_wheel_joint" type="continuous">
-    <parent link="base_link" />
-    <child link="left_wheel" />
-    <origin xyz="0.25 0.13 -0.1" rpy="-${pi/2} 0 0" />
-    <axis xyz="0 0 1" />
-  </joint>
-  <link name="left_wheel">
-    <visual>
-      <origin xyz="0 0 0" rpy="-${pi/2} 0 0" />
-      <geometry>
-        <!--The
-        package resolves into install/forklift_controller/share/forklift_controller/-->
-        <mesh filename="package://forklift_controller/models/forklift/meshes/front_wheel_right.dae"
-          scale="0.0025 0.0025 0.0025" />
-      </geometry>
-    </visual>
-    <collision>
-      <origin xyz="0 0 0" rpy="0 0 0" />
-      <geometry>
-        <cylinder radius="0.08" length="0.02" />
-      </geometry>
-    </collision>
-    <xacro:inertial_cylinder mass="5" length="0.02" radius="0.08">
-      <origin xyz="0 0 0" rpy="0 0 0" />
-    </xacro:inertial_cylinder>
-  </link>
-  <!-- RIGHT WHEEL LINK -->
-  <joint name="right_wheel_joint" type="continuous">
-    <parent link="base_link" />
-    <child link="right_wheel" />
-    <origin xyz="0.25 -0.13 -0.1" rpy="-${pi/2} 0 0" />
-    <axis xyz="0 0 1" />
-  </joint>
-  <link name="right_wheel">
-    <visual>
-      <origin xyz="0 0 0" rpy="${pi/2} 0 0" />
-      <geometry>
-        <!-- package://forklift_controller resolves to
-        install/forklift_controller/share/forklift_controller-->
-        <mesh filename="package://forklift_controller/models/forklift/meshes/front_wheel_right.dae"
-          scale="0.0025 0.0025 0.0025" />
-      </geometry>
-    </visual>
-    <collision>
-      <origin xyz="0 0 0" rpy="0 0 0" />
-      <geometry>
-        <cylinder radius="0.08" length="0.02" />
-      </geometry>
-    </collision>
-    <xacro:inertial_cylinder mass="5" length="0.02" radius="0.08">
-      <origin xyz="0 0 0" rpy="0 0 0" />
-    </xacro:inertial_cylinder>
-  </link>
+  <xacro:fork id="1" mass="15" scale="1" fork_attach_offsets="0.05 0.2 -0.35"></xacro:fork>
+  <xacro:fork id="2" mass="15" scale="1" fork_attach_offsets="0.05 -0.2 -0.35"></xacro:fork>
+  <xacro:wheel name="right_wheel" mass="5" scale="1" x="0.8" y="-0.4" z="-0.35" roll="0"></xacro:wheel>
+  <xacro:wheel name="right_wheel_back" mass="5" scale="1" x="-0.65" y="-0.4" z="-0.35" roll="0"></xacro:wheel>
+  <xacro:wheel name="left_wheel" mass="5" scale="1" x="0.8" y="0.4" z="-0.35" roll="${pi}"></xacro:wheel>
+  <xacro:wheel name="left_wheel_back" mass="5" scale="1" x="-0.65" y="0.4" z="-0.35" roll="${pi}"></xacro:wheel>
   <gazebo>
     <!--
@@ -204,52 +153,4 @@
     <preserveFixedJoint>true</preserveFixedJoint>
   </gazebo>
-  <joint name="right_wheel_back_joint" type="continuous">
-    <parent link="base_link" />
-    <child link="right_wheel_back" />
-    <origin xyz="-0.2 -0.13 -0.1" rpy="-${pi/2} 0 0" />
-    <axis xyz="0 0 1" />
-  </joint>
-  <link name="right_wheel_back">
-    <visual>
-      <origin xyz="0 0 0" rpy="${pi/2} 0 0" />
-      <geometry>
-        <mesh filename="package://forklift_controller/models/forklift/meshes/front_wheel_right.dae"
-          scale="0.0025 0.0025 0.0025" />
-      </geometry>
-    </visual>
-    <collision>
-      <origin xyz="0 0 0" rpy="0 0 0" />
-      <geometry>
-        <cylinder radius="0.08" length="0.02" />
-      </geometry>
-    </collision>
-    <xacro:inertial_cylinder mass="5" length="0.02" radius="0.08">
-      <origin xyz="0 0 0" rpy="0 0 0" />
-    </xacro:inertial_cylinder>
-  </link>
-  <joint name="left_wheel_back_joint" type="continuous">
-    <parent link="base_link" />
-    <child link="left_wheel_back" />
-    <origin xyz="-0.2 0.13 -0.1" rpy="-${pi/2} 0 0" />
-    <axis xyz="0 0 1" />
-  </joint>
-  <link name="left_wheel_back">
-    <visual>
-      <origin xyz="0 0 0" rpy="-${pi/2} 0 0" />
-      <geometry>
-        <mesh filename="package://forklift_controller/models/forklift/meshes/front_wheel_right.dae"
-          scale="0.0025 0.0025 0.0025" />
-      </geometry>
-    </visual>
-    <collision>
-      <origin xyz="0 0 0" rpy="0 0 0" />
-      <geometry>
-        <cylinder radius="0.08" length="0.02" />
-      </geometry>
-    </collision>
-    <xacro:inertial_cylinder mass="5" length="0.02" radius="0.08">
-      <origin xyz="0 0 0" rpy="0 0 0" />
-    </xacro:inertial_cylinder>
-  </link>
   <!--
   <gazebo reference="fork_plate_joint">
