Commit message: Somewhat working version of nav

File: src/forklift_controller/urdf/robot.urdf.xacro (robot description, xacro)
@@ -8,13 +8,17 @@
         name="gz::sim::systems::DiffDrive">
             <left_joint>left_wheel_joint</left_joint>
-            <left_joint>left_wheel_back_joint</left_joint>
+            <!-- <left_joint>left_wheel_back_joint</left_joint> -->
             <right_joint>right_wheel_joint</right_joint>
-            <right_joint>right_wheel_back_joint</right_joint>
+            <!-- <right_joint>right_wheel_back_joint</right_joint> -->
             <wheel_separation>0.3</wheel_separation>
             <wheel_radius>0.07</wheel_radius>
-            <odom_publish_frequency>1</odom_publish_frequency>
-            <odom_topic>pos</odom_topic>
-            <topic>$(arg robot_namespace)/cmd_vel</topic>
+            <odom_publish_frequency>30</odom_publish_frequency>
+            <odom_topic>/odom</odom_topic>
+            <frame_id>odom</frame_id>
+            <tf_topic>tf</tf_topic>
+            <topic>/cmd_vel</topic>
+            <child_frame_id>base_link</child_frame_id>
         </plugin>
+        <!--
         <plugin
         filename="gz-sim-odometry-publisher-system"
@@ -23,5 +27,4 @@
             <odom_topic>$(arg robot_namespace)/odometry</odom_topic>
         </plugin>
-        <!--
         <plugin
             filename="gz-sim-pose-publisher-system"
@@ -34,5 +37,10 @@
         -->
       <plugin filename="gz-sim-joint-state-publisher-system" name="gz::sim::systems::JointStatePublisher">
-          <topic>$(arg robot_namespace)/joint_states</topic>
+        <topic>joint_states</topic>
+        <joint_name>left_wheel_joint</joint_name>
+        <joint_name>right_wheel_joint</joint_name>
+        <joint_name>left_wheel_back_joint</joint_name>
+        <joint_name>right_wheel_back_joint</joint_name>
+          <!-- <topic>$(arg robot_namespace)/joint_states</topic> -->
       </plugin>
       <plugin filename="gz-sim-joint-position-controller-system" name="gz::sim::systems::JointPositionController">

File: src/forklift_controller/urdf/robot_core.xacro (robot description, xacro)
@@ -21,13 +21,24 @@
     <xacro:property name="base_width" value="0.3"/>
     <link name="base_footprint">
+        <inertial>
+            <mass value="0.0001"/>
+            <origin xyz="0 0 0"/>
+            <inertia ixx="0.0001" ixy="0.0" ixz="0.0" iyy="0.0001" iyz="0.0" izz="0.0001"/>
+          </inertial>
+          <visual>
+            <origin rpy="0 0 0" xyz="0 0 0"/>
+            <geometry>
+              <box size="0.001 0.001 0.001"/>
+            </geometry>
+          </visual>
     </link>
     <joint name="base_link_joint" type="fixed">
         <parent link="base_link"/>
         <child link="base_footprint"/>
-        <origin xyz="0 0 0" rpy="0 0 0"/>
+        <origin xyz="0 0 -0.15" rpy="0 0 0"/>
     </joint>
     <link name="base_link">
         <visual>
-            <origin xyz="0 0 0.05"/>
+            <origin xyz="0 0 0"/>
             <geometry>
                 <mesh filename="$(find forklift_controller)/meshes/body.dae" scale="0.0027 0.0027 0.0027"/>
@@ -37,5 +48,6 @@
             <origin xyz="0 0 0"/>
             <geometry>
-                <box size="0.3 ${base_width} ${base_height}"/>
+                <mesh filename="$(find forklift_controller)/meshes/body.dae" scale="0.0027 0.0027 0.0027"/>
+                <!-- <box size="0.3 ${base_width} ${base_height}"/> -->
             </geometry>
         </collision>
@@ -118,17 +130,50 @@
         <parent link="fork_plate"/>
         <child link="fork_2"/>
-        <!--Offset the joint position by the track depth amount-->
         <origin xyz="0 0.05 -0.01" rpy="0 0 0"/>
     </joint>
+     <!--Offset the joint position by the track depth amount-->
+    <!--
+    <joint name="caster" type="fixed">
+        <parent link="base_link"/>
+        <child link="caster_link"/>
+        <origin rpy="0 0 0" xyz="-0.15 0 -0.10"/>
+      </joint>
+      <link name="caster_link">
+        <visual>
+          <origin rpy="0 0 0" xyz="0 0 0"/>
+          <geometry>
+            <sphere radius="0.05"/>
+          </geometry>
+        </visual>
+        <collision>
+          <origin rpy="0 0 0" xyz="0 0 0"/>
+          <geometry>
+            <sphere radius="0.05"/>
+          </geometry>
+        </collision>
+        <inertial>
+          <mass value="0.1"/>
+          <origin rpy="0 0 0" xyz="0 0 0"/>
+          <inertia ixx="0.0001" ixy="0" ixz="0" iyy="0.0001" iyz="0" izz="0.0001"/>
+        </inertial>
+      </link>
+      <gazebo reference="caster_link">
+        <material>Gazebo/DarkGrey</material>
+        <mu1>0.1</mu1>
+        <mu2>0.1</mu2>
+        <kp>1000000.0</kp>
+        <kd>1.0</kd>
+      </gazebo>
+    -->
     <!-- LEFT WHEEL LINK -->
     <joint name="left_wheel_joint" type="continuous">
         <parent link="base_link"/>
         <child link="left_wheel"/>
-        <origin xyz="0.23 0.13 -0.075" rpy="0 0 0" />
-        <axis xyz="0 1 0"/>
+        <origin xyz="0.23 0.13 -0.075" rpy="-${pi/2} 0 0" />
+        <axis xyz="0 0 1"/>
     </joint>
     <link name="left_wheel">
         <visual>
-            <origin xyz="0 0 0" rpy="0 0 0"/>
+            <origin xyz="0 0 0" rpy="-${pi/2} 0 0"/>
             <geometry>
                 <mesh filename="$(find forklift_controller)/meshes/front_wheel_right.dae" scale="0.002 0.002 0.002"/>
@@ -136,5 +181,5 @@
         </visual>
         <collision>
-            <origin xyz="0 0 0" rpy="-${pi/2} 0 0"/>
+            <origin xyz="0 0 0" rpy="0 0 0"/>
             <geometry>
                 <cylinder radius="0.07" length="0.02"/>
@@ -143,28 +188,4 @@
         <xacro:inertial_cylinder mass="0.1" length="0.02" radius="0.05">
             <origin xyz="0 0 0" rpy="0 0 0"/>
-        </xacro:inertial_cylinder>
-    </link>
-    <joint name="left_wheel_back_joint" type="continuous">
-        <parent link="base_link"/>
-        <child link="left_wheel_back"/>
-        <origin xyz="-0.2 0.13 -0.075" rpy="0 0 0" />
-        <axis xyz="0 1 0"/>
-    </joint>
-    <link name="left_wheel_back">
-        <visual>
-            <origin xyz="0 0 0" rpy="0 0 ${pi}"/>
-            <geometry>
-                <mesh filename="$(find forklift_controller)/meshes/front_wheel_right.dae" scale="0.002 0.002 0.002"/>
-                <!-- <cylinder radius="0.05" length="0.02"/> -->
-            </geometry>
-        </visual>
-        <collision>
-            <origin xyz="0 0 0" rpy="-${pi/2} 0 0"/>
-            <geometry>
-                <cylinder radius="0.07" length="0.02"/>
-            </geometry>
-        </collision>
-        <xacro:inertial_cylinder mass="0.1" length="0.02" radius="0.05">
-            <origin xyz="0 0 0" rpy="-${pi/2} 0 0"/>
         </xacro:inertial_cylinder>
     </link>
@@ -173,10 +194,10 @@
         <parent link="base_link"/>
         <child link="right_wheel"/>
-        <origin xyz="0.23 -0.13 -0.075" rpy="0 0 0" />
-        <axis xyz="0 1 0"/>
+        <origin xyz="0.23 -0.13 -0.075" rpy="-${pi/2} 0 0" />
+        <axis xyz="0 0 1"/>
     </joint>
     <link name="right_wheel">
         <visual>
-            <origin xyz="0 0 0" rpy="0 0 0"/>
+            <origin xyz="0 0 0" rpy="${pi/2} 0 0"/>
             <geometry>
                 <mesh filename="$(find forklift_controller)/meshes/front_wheel_right.dae" scale="0.002 0.002 0.002"/>
@@ -184,5 +205,5 @@
         </visual>
         <collision>
-            <origin xyz="0 0 0" rpy="-${pi/2} 0 0"/>
+            <origin xyz="0 0 0" rpy="0 0 0"/>
             <geometry>
                 <cylinder radius="0.07" length="0.02"/>
@@ -190,27 +211,5 @@
         </collision>
         <xacro:inertial_cylinder mass="0.1" length="0.02" radius="0.05">
-            <origin xyz="0 0 0" rpy="-${pi/2} 0 0"/>
-        </xacro:inertial_cylinder>
-    </link>
-    <joint name="right_wheel_back_joint" type="continuous">
-        <parent link="base_link"/>
-        <child link="right_wheel_back"/>
-        <origin xyz="-0.2 -0.13 -0.075" rpy="0 0 0" />
-        <axis xyz="0 1 0"/>
-    </joint>
-    <link name="right_wheel_back">
-        <visual>
-            <geometry>
-                <mesh filename="$(find forklift_controller)/meshes/front_wheel_right.dae" scale="0.002 0.002 0.002"/>
-            </geometry>
-        </visual>
-        <collision>
-            <origin xyz="0 0 0" rpy="-${pi/2} 0 0"/>
-            <geometry>
-                <cylinder radius="0.07" length="0.02"/>
-            </geometry>
-        </collision>
-        <xacro:inertial_cylinder mass="0.1" length="0.02" radius="0.05">
-            <origin xyz="0 0 0" rpy="-${pi/2} 0 0"/>
+            <origin xyz="0 0 0" rpy="0 0 0"/>
         </xacro:inertial_cylinder>
     </link>
@@ -230,33 +229,167 @@
                     </contact>
             </sensor>
-        </gazebo>
-    <gazebo reference="base_link">
-    <sensor name="lidar" type="gpu_lidar">
-      <!-- <gz_frame_id>fork_plate_fixed_joint_lump__fork_1_collision_1</gz_frame_id> -->
-      <topic>scan</topic>
+    </gazebo>
+    <link name="rplidar_link">
+        <visual>
+            <origin xyz="0 0 0" rpy="0 0 0"/>
+            <geometry>
+                <box size="0.01 0.1 0.2"/>
+            </geometry>
+        </visual>
+        <collision>
+            <origin xyz="0 0 0" rpy="0 0 0"/>
+            <geometry>
+                <box size="0.01 0.3 0.2"/>
+            </geometry>
+        </collision>
+        <inertial>
+            <mass value="75"/>
+            <origin xyz="0.005 0.15 0.1" rpy="0 0 0"/>
+            <inertia ixx="0.075" ixy="0" ixz="0" iyy="0.075" iyz="0" izz="0.0045"/>
+        </inertial>
+    </link>
+    <joint name="rplidar_joint" type="fixed">
+        <parent link="base_link"/>
+        <child link="rplidar_link"/>
+        <origin xyz="0 0 0.5" rpy="0 0 0"/>
+    </joint>
+    <gazebo reference="rplidar_link">
+        <sensor name="rplidar" type="gpu_lidar">
+          <update_rate>10.0</update_rate>
+          <visualize>true</visualize>
+          <always_on>true</always_on>
+          <gz_frame_id>rplidar_link</gz_frame_id>
+          <topic>scan</topic>
+          <lidar>
+            <scan>
+              <horizontal>
+                <samples>360</samples>
+                <resolution>1.0</resolution>
+                <min_angle>0.000</min_angle>
+                <max_angle>6.280000</max_angle>
+              </horizontal>
+            </scan>
+            <range>
+              <min>0.164</min>
+              <max>20.0</max>
+              <resolution>0.01</resolution>
+            </range>
+          </lidar>
+          <plugin name="dummy" filename="dummyfile"></plugin>
+        </sensor>
+      </gazebo>
+  <gazebo reference="rplidar_joint">
+    <preserveFixedJoint>true</preserveFixedJoint>
+  </gazebo>
+      <joint name="right_wheel_back_joint" type="continuous">
+        <parent link="base_link"/>
+        <child link="right_wheel_back"/>
+        <origin xyz="-0.2 -0.13 -0.075" rpy="-${pi/2} 0 0" />
+        <axis xyz="0 0 1"/>
+    </joint>
+    <link name="right_wheel_back">
+        <visual>
+            <origin xyz="0 0 0" rpy="${pi/2} 0 0"/>
+            <geometry>
+                <mesh filename="$(find forklift_controller)/meshes/front_wheel_right.dae" scale="0.002 0.002 0.002"/>
+            </geometry>
+        </visual>
+        <collision>
+            <origin xyz="0 0 0" rpy="0 0 0"/>
+            <geometry>
+                <cylinder radius="0.07" length="0.02"/>
+            </geometry>
+        </collision>
+        <xacro:inertial_cylinder mass="0.1" length="0.02" radius="0.05">
+            <origin xyz="0 0 0" rpy="0 0 0"/>
+        </xacro:inertial_cylinder>
+    </link>
+      <joint name="left_wheel_back_joint" type="continuous">
+        <parent link="base_link"/>
+        <child link="left_wheel_back"/>
+        <origin xyz="-0.2 0.13 -0.075" rpy="-${pi/2} 0 0" />
+        <axis xyz="0 0 1"/>
+    </joint>
+    <link name="left_wheel_back">
+        <visual>
+            <origin xyz="0 0 0" rpy="-${pi/2} 0 0"/>
+            <geometry>
+                <mesh filename="$(find forklift_controller)/meshes/front_wheel_right.dae" scale="0.002 0.002 0.002"/>
+            </geometry>
+        </visual>
+        <collision>
+            <origin xyz="0 0 0" rpy="0 0 0"/>
+            <geometry>
+                <cylinder radius="0.07" length="0.02"/>
+            </geometry>
+        </collision>
+        <xacro:inertial_cylinder mass="0.1" length="0.02" radius="0.05">
+            <origin xyz="0 0 0" rpy="0 0 0"/>
+        </xacro:inertial_cylinder>
+    </link>
+    <!--Make the back wheel almost frictionless in order to simulate free wheels-->
+    <gazebo reference="left_wheel_back">
+        <mu1>0.1</mu1>
+        <mu2>0.1</mu2>
+        <kp>1000000.0</kp>
+        <kd>1.0</kd>
+      </gazebo>
+      <gazebo reference="right_wheel_back">
+        <mu1>0.1</mu1>
+        <mu2>0.1</mu2>
+        <kp>1000000.0</kp>
+        <kd>1.0</kd>
+      </gazebo>
+      <!--
+  <gazebo reference="base_link">
+    <sensor type="imu" name="imu_sensor">
+      <preserveFixedJoint>true</preserveFixedJoint>
       <always_on>true</always_on>
-      <visualize>true</visualize>
-      <update_rate>5</update_rate>
-      <ray>
-        <scan>
-          <horizontal>
-            <samples>360</samples>
-            <resolution>1.000000</resolution>
-            <min_angle>0.000000</min_angle>
-            <max_angle>6.280000</max_angle>
-          </horizontal>
-        </scan>
-        <range>
-          <min>0.120000</min>
-          <max>1.0</max>
-          <resolution>0.015000</resolution>
-        </range>
-        <noise>
-          <type>gaussian</type>
-          <mean>0.0</mean>
-          <stddev>0.01</stddev>
-        </noise>
-      </ray>
+      <update_rate>30</update_rate>
+      <topic>imu</topic>
+      <imu>
+        <angular_velocity>
+          <x>
+            <noise type="gaussian">
+              <mean>0.0</mean>
+              <stddev>0.0</stddev>
+            </noise>
+          </x>
+          <y>
+            <noise type="gaussian">
+              <mean>0.0</mean>
+              <stddev>0.0</stddev>
+            </noise>
+          </y>
+          <z>
+            <noise type="gaussian">
+              <mean>0.0</mean>
+              <stddev>0.0</stddev>
+            </noise>
+          </z>
+        </angular_velocity>
+        <linear_acceleration>
+          <x>
+            <noise type="gaussian">
+              <mean>0.0</mean>
+              <stddev>0.0</stddev>
+            </noise>
+          </x>
+          <y>
+            <noise type="gaussian">
+              <mean>0.0</mean>
+              <stddev>0.0</stddev>
+            </noise>
+          </y>
+          <z>
+            <noise type="gaussian">
+              <mean>0.0</mean>
+              <stddev>0.0</stddev>
+            </noise>
+          </z>
+        </linear_acceleration>
+      </imu>
     </sensor>
   </gazebo>
+    -->
 </robot>

Commit message: Improve robot collision

File: src/forklift_controller/urdf/robot.urdf.xacro (robot description, xacro)
@@ -43,4 +43,5 @@
         <topic>$(arg namespace)/joint_states</topic>
       </plugin>
+      <!--
       <plugin filename="gz-sim-joint-position-controller-system" name="gz::sim::systems::JointPositionController">
         <joint_name>fork_plate_joint</joint_name>
@@ -48,4 +49,5 @@
         <initial_position>0.6</initial_position>
       </plugin>
+      -->
     </gazebo>
 </robot>

File: src/forklift_controller/urdf/robot_core.xacro (robot description, xacro)
@@ -73,5 +73,5 @@
         <inertial>
             <mass value="75"/>
-            <origin xyz="0.005 0.15 0.1" rpy="0 0 0"/>
+            <origin xyz="0 0 0" rpy="0 0 0"/>
             <inertia ixx="0.075" ixy="0" ixz="0" iyy="0.075" iyz="0" izz="0.0045"/>
         </inertial>
@@ -81,5 +81,5 @@
         <child link="fork_plate"/>
         <!--Offset the joint position by the track depth amount-->
-        <origin xyz="0.375 0 0" rpy="0 0 0"/>
+        <origin xyz="0.375 0 0.05" rpy="0 0 0"/>
         <axis xyz="0 0 1"/>
         <limit effort="110" lower="0" upper="0.6" velocity="0.5"/>
@@ -87,5 +87,5 @@
     <link name="fork_1">
         <visual>
-            <origin xyz="0 0.02 0" rpy="0 0 -${pi}"/>
+            <origin xyz="0 0 0" rpy="0 0 -${pi}"/>
             <geometry>
                 <mesh filename="$(find forklift_controller)/models/forklift/meshes/fork.dae" scale="0.0027 0.0027 0.0027"/>
@@ -102,5 +102,5 @@
         <inertial>
             <mass value="50"/>
-            <origin xyz="0.15 0 0" rpy="0 0 0"/>
+            <origin xyz="0 0 0" rpy="0 0 0"/>
             <inertia ixx="0.00010417" ixy="0" ixz="0" iyy="0.06510417" iyz="0" izz="0.06510417"/>
         </inertial>
@@ -114,5 +114,5 @@
         <visual>
             <!-- For some reason, the another forks origin is a bit different than fork1-->
-            <origin xyz="0 0.01 0" rpy="0 0 -${pi}"/>
+            <origin xyz="0 0 0" rpy="0 0 -${pi}"/>
             <geometry>
               <mesh filename="$(find forklift_controller)/models/forklift/meshes/fork.dae" scale="0.0027 0.0027 0.0027"/>
@@ -127,5 +127,5 @@
         <inertial>
             <mass value="50"/>
-            <origin xyz="0.15 0 0" rpy="0 0 0"/>
+            <origin xyz="0 0 0" rpy="0 0 0"/>
             <inertia ixx="0.00010417" ixy="0" ixz="0" iyy="0.06510417" iyz="0" izz="0.06510417"/>
         </inertial>
@@ -288,5 +288,5 @@
         <parent link="base_link"/>
         <child link="right_wheel_back"/>
-        <origin xyz="-0.2 -0.13 -0.075" rpy="-${pi/2} 0 0" />
+        <origin xyz="-0.2 -0.13 -0.1" rpy="-${pi/2} 0 0" />
         <axis xyz="0 0 1"/>
     </joint>
@@ -301,5 +301,5 @@
             <origin xyz="0 0 0" rpy="0 0 0"/>
             <geometry>
-                <cylinder radius="0.07" length="0.02"/>
+                <cylinder radius="0.065" length="0.02"/>
             </geometry>
         </collision>
@@ -311,5 +311,5 @@
         <parent link="base_link"/>
         <child link="left_wheel_back"/>
-        <origin xyz="-0.2 0.13 -0.075" rpy="-${pi/2} 0 0" />
+        <origin xyz="-0.2 0.13 -0.1" rpy="-${pi/2} 0 0" />
         <axis xyz="0 0 1"/>
     </joint>
@@ -324,5 +324,5 @@
             <origin xyz="0 0 0" rpy="0 0 0"/>
             <geometry>
-                <cylinder radius="0.07" length="0.02"/>
+                <cylinder radius="0.065" length="0.02"/>
             </geometry>
         </collision>
