Commit message: Implement 4-wheeled drive

File: src/forklift_controller/urdf/robot.urdf.xacro (robot description, xacro)
@@ -8,8 +8,8 @@
         name="gz::sim::systems::DiffDrive">
             <left_joint>left_wheel_joint</left_joint>
-            <!-- <left_joint>left_wheel_back_joint</left_joint> -->
+            <left_joint>left_wheel_back_joint</left_joint>
             <right_joint>right_wheel_joint</right_joint>
-            <!-- <right_joint>right_wheel_back_joint</right_joint> -->
-            <wheel_separation>0.3</wheel_separation>
+            <right_joint>right_wheel_back_joint</right_joint>
+            <wheel_separation>0.26</wheel_separation>
             <wheel_radius>0.07</wheel_radius>
             <odom_publish_frequency>30</odom_publish_frequency>
@@ -19,4 +19,12 @@
             <topic>$(arg namespace)/cmd_vel</topic>
             <child_frame_id>base_link</child_frame_id>
+            <max_linear_acceleration>10</max_linear_acceleration>
+            <min_linear_acceleration>-10</min_linear_acceleration>
+            <max_angular_acceleration>20</max_angular_acceleration>
+            <min_angular_acceleration>-20</min_angular_acceleration>
+            <max_linear_velocity>0.5</max_linear_velocity>
+            <min_linear_velocity>-0.5</min_linear_velocity>
+            <max_angular_velocity>10</max_angular_velocity>
+            <min_angular_velocity>-10</min_angular_velocity>
         </plugin>
         <!--

File: src/forklift_controller/urdf/robot_core.xacro (robot description, xacro)
@@ -19,6 +19,15 @@
     <xacro:property name="track_depth" value="0.02"/> <!--This is actually the depth of the track when in up position-->
     <xacro:property name="track_width" value="0.05"/> <!--This is actually the depth of the track when in up position-->
-    <xacro:property name="base_height" value="0.15"/>
+    <xacro:property name="base_height" value="0.52"/>
     <xacro:property name="base_width" value="0.3"/>
+    <xacro:property name="base_length" value="0.68"/>
+    <xacro:property name="fork_mass" value="15"/>
+    <!--Simple collision calculation, used for inertia-->
+    <!--
+      <origin xyz="0.042 0 0.14"/>
+            <geometry>
+              <box size="${base_length} ${base_width} ${base_height}"/>
+            </geometry>
+    -->
     <link name="base_footprint">
         <inertial>
@@ -47,12 +56,15 @@
         </visual>
         <collision>
-            <origin xyz="0 0 0"/>
-            <geometry>
+            <origin xyz="0.042 0 0.14"/>
+            <geometry>
+              <!--
                 <mesh filename="$(find forklift_controller)/models/forklift/meshes/body.dae"
                   scale="${scaler*0.0027} ${scaler*0.0027} ${scaler*0.0027}"/>
-            </geometry>
-        </collision>
-        <xacro:inertial_box mass="500" x="0.3" y="${base_width}" z="${base_height}">
-            <origin xyz="0 0 0" rpy="0 0 0"/>
+                -->
+              <box size="${base_length} ${base_width} ${base_height}"/>
+            </geometry>
+        </collision>
+        <xacro:inertial_box mass="50" x="${base_length}" y="${base_width}" z="${base_height}">
+            <origin xyz="-0.1 0 0" rpy="0 0 0"/>
         </xacro:inertial_box>
     </link>
@@ -61,5 +73,4 @@
             <origin xyz="0 0 0" rpy="0 0 0"/>
             <geometry>
-                <!-- <box size="0.01 0.2 0.2"/> -->
                 <mesh filename="$(find forklift_controller)/models/forklift/meshes/fork_plate.dae" scale="0.0027 0.0027 0.0027"/>
             </geometry>
@@ -71,14 +82,11 @@
             </geometry>
         </collision>
-        <inertial>
-            <mass value="75"/>
-            <origin xyz="0 0 0" rpy="0 0 0"/>
-            <inertia ixx="0.075" ixy="0" ixz="0" iyy="0.075" iyz="0" izz="0.0045"/>
-        </inertial>
+          <xacro:inertial_box mass="50" x="0.01" y="0.3" z="0.2">
+            <origin xyz="0 0 0" rpy="0 0 0"/>
+        </xacro:inertial_box>
     </link>
     <joint name="fork_plate_joint" type="fixed">
         <parent link="base_link"/>
         <child link="fork_plate"/>
-        <!--Offset the joint position by the track depth amount-->
         <origin xyz="0.375 0 0.05" rpy="0 0 0"/>
         <axis xyz="0 0 1"/>
@@ -86,24 +94,28 @@
     </joint>
     <link name="fork_1">
-        <visual>
-            <origin xyz="0 0 0" rpy="0 0 -${pi}"/>
-            <geometry>
-                <mesh filename="$(find forklift_controller)/models/forklift/meshes/fork.dae" scale="0.0027 0.0027 0.0027"/>
-                <!-- <box size="0.3 0.05 0.01"/> -->
-            </geometry>
-        </visual>
-        <collision>
-            <origin xyz="0 0 0"  rpy="0 0 -${pi}"/>
-            <geometry>
-                <mesh filename="$(find forklift_controller)/models/forklift/meshes/fork.dae" scale="0.0027 0.0027 0.0027"/>
-                <!-- <box size="0.3 0.05 0.01"/> -->
-            </geometry>
-        </collision>
-        <inertial>
-            <mass value="50"/>
-            <origin xyz="0 0 0" rpy="0 0 0"/>
-            <inertia ixx="0.00010417" ixy="0" ixz="0" iyy="0.06510417" iyz="0" izz="0.06510417"/>
-        </inertial>
-    </link>
+      <visual>
+          <origin xyz="0 0 0" rpy="0 0 -${pi}"/>
+          <geometry>
+              <mesh filename="$(find forklift_controller)/models/forklift/meshes/fork.dae" scale="0.0027 0.0027 0.0027"/>
+          </geometry>
+      </visual>
+      <collision>
+          <origin xyz="0 0 0"  rpy="0 0 -${pi}"/>
+          <geometry>
+              <mesh filename="$(find forklift_controller)/models/forklift/meshes/fork.dae" scale="0.0027 0.0027 0.0027"/>
+          </geometry>
+      </collision>
+      <inertial>
+          <origin xyz="-0.03808040868302371, 0.00482172099079702, -0.016262899934648207"></origin>
+          <mass value="${fork_mass}"/>
+          <inertia
+          ixx="${2.55322 * fork_mass * (0.0027**5)}"
+          ixy="${2.05649 * fork_mass * (0.0027**5)}"
+          ixz="${-2.66481 * fork_mass * (0.0027**5)}"
+          iyy="${11.5514 * fork_mass * (0.0027**5)}"
+          iyz="${1.45586  * fork_mass * (0.0027**5)}"
+          izz="${9.14891 * fork_mass * (0.0027**5)}" />
+      </inertial>
+  </link>
     <joint name="fork_1_joint" type="fixed">
         <parent link="fork_plate"/>
@@ -111,7 +123,7 @@
         <origin xyz="-0.02 -0.06 -0.07" rpy="0 0 0"/>
     </joint>
+    <!--
     <link name="fork_2">
         <visual>
-            <!-- For some reason, the another forks origin is a bit different than fork1-->
             <origin xyz="0 0 0" rpy="0 0 -${pi}"/>
             <geometry>
@@ -126,7 +138,9 @@
         </collision>
         <inertial>
-            <mass value="50"/>
-            <origin xyz="0 0 0" rpy="0 0 0"/>
-            <inertia ixx="0.00010417" ixy="0" ixz="0" iyy="0.06510417" iyz="0" izz="0.06510417"/>
+            <mass value="${fork_mass}"/>
+            <inertia
+            ixx="${1.27661 * fork_mass}" ixy="${1.028245 * fork_mass}" ixz="${-1.332405 * fork_mass}"
+            iyy="${5.7757 * fork_mass}" iyz="${0.72793 * fork_mass}"
+            izz="${4.574455 * fork_mass}" />
         </inertial>
     </link>
@@ -136,4 +150,5 @@
         <origin xyz="-0.02 0.06 -0.07" rpy="0 0 0"/>
     </joint>
+    -->
      <!--Offset the joint position by the track depth amount-->
     <!--
@@ -174,5 +189,5 @@
         <parent link="base_link"/>
         <child link="left_wheel"/>
-        <origin xyz="0.23 0.13 -0.075" rpy="-${pi/2} 0 0" />
+        <origin xyz="0.23 0.13 -0.1" rpy="-${pi/2} 0 0" />
         <axis xyz="0 0 1"/>
     </joint>
@@ -187,8 +202,8 @@
             <origin xyz="0 0 0" rpy="0 0 0"/>
             <geometry>
-                <cylinder radius="0.07" length="0.02"/>
-            </geometry>
-        </collision>
-        <xacro:inertial_cylinder mass="0.1" length="0.02" radius="0.05">
+                <cylinder radius="0.08" length="0.02"/>
+            </geometry>
+        </collision>
+        <xacro:inertial_cylinder mass="5" length="0.02" radius="0.08">
             <origin xyz="0 0 0" rpy="0 0 0"/>
         </xacro:inertial_cylinder>
@@ -198,5 +213,5 @@
         <parent link="base_link"/>
         <child link="right_wheel"/>
-        <origin xyz="0.23 -0.13 -0.075" rpy="-${pi/2} 0 0" />
+        <origin xyz="0.23 -0.13 -0.1" rpy="-${pi/2} 0 0" />
         <axis xyz="0 0 1"/>
     </joint>
@@ -211,8 +226,8 @@
             <origin xyz="0 0 0" rpy="0 0 0"/>
             <geometry>
-                <cylinder radius="0.07" length="0.02"/>
-            </geometry>
-        </collision>
-        <xacro:inertial_cylinder mass="0.1" length="0.02" radius="0.05">
+                <cylinder radius="0.08" length="0.02"/>
+            </geometry>
+        </collision>
+        <xacro:inertial_cylinder mass="5" length="0.02" radius="0.08">
             <origin xyz="0 0 0" rpy="0 0 0"/>
         </xacro:inertial_cylinder>
@@ -301,8 +316,8 @@
             <origin xyz="0 0 0" rpy="0 0 0"/>
             <geometry>
-                <cylinder radius="0.065" length="0.02"/>
-            </geometry>
-        </collision>
-        <xacro:inertial_cylinder mass="0.1" length="0.02" radius="0.05">
+                <cylinder radius="0.08" length="0.02"/>
+            </geometry>
+        </collision>
+        <xacro:inertial_cylinder mass="5" length="0.02" radius="0.08">
             <origin xyz="0 0 0" rpy="0 0 0"/>
         </xacro:inertial_cylinder>
@@ -324,8 +339,8 @@
             <origin xyz="0 0 0" rpy="0 0 0"/>
             <geometry>
-                <cylinder radius="0.065" length="0.02"/>
-            </geometry>
-        </collision>
-        <xacro:inertial_cylinder mass="0.1" length="0.02" radius="0.05">
+                <cylinder radius="0.08" length="0.02"/>
+            </geometry>
+        </collision>
+        <xacro:inertial_cylinder mass="5" length="0.02" radius="0.08">
             <origin xyz="0 0 0" rpy="0 0 0"/>
         </xacro:inertial_cylinder>
@@ -333,14 +348,102 @@
     <!--Make the back wheel almost frictionless in order to simulate free wheels-->
     <gazebo reference="left_wheel_back">
-        <mu1>0.1</mu1>
-        <mu2>0.1</mu2>
-        <kp>1000000.0</kp>
-        <kd>1.0</kd>
+      <friction>
+        <ode>
+          <mu>1.01</mu>
+          <mu2>1.01</mu2>
+          <fdir1>0 0 1</fdir1>
+          <slip1>0</slip1>
+          <slip2>0</slip2>
+        </ode>
+      </friction>
+      <bounce>
+        <restitution_coefficient>0.0</restitution_coefficient>
+        <threshold>100000.0</threshold>
+      </bounce>
+      <contact>
+        <ode>
+          <soft_cfm>0.0</soft_cfm>
+          <soft_erp>0.2</soft_erp>
+          <kp>100000.0</kp>
+          <kd>1.0</kd>
+          <max_vel>100.0</max_vel>
+          <min_depth>0.001</min_depth>
+        </ode>
+      </contact>
+      </gazebo>
+      <gazebo reference="left_wheel">
+        <friction>
+          <ode>
+            <mu>1.01</mu>
+            <mu2>1.01</mu2>
+            <fdir1>0 0 1</fdir1>
+            <slip1>0</slip1>
+            <slip2>0</slip2>
+          </ode>
+        </friction>
+        <bounce>
+          <restitution_coefficient>0.0</restitution_coefficient>
+          <threshold>100000.0</threshold>
+        </bounce>
+        <contact>
+          <ode>
+            <soft_cfm>0.0</soft_cfm>
+            <soft_erp>0.2</soft_erp>
+            <kp>100000.0</kp>
+            <kd>1.0</kd>
+            <max_vel>100.0</max_vel>
+            <min_depth>0.001</min_depth>
+          </ode>
+        </contact>
+      </gazebo>
+      <gazebo reference="right_wheel">
+        <friction>
+          <ode>
+            <mu>1.01</mu>
+            <mu2>1.01</mu2>
+            <fdir1>0 0 1</fdir1>
+            <slip1>0</slip1>
+            <slip2>0</slip2>
+          </ode>
+        </friction>
+        <bounce>
+          <restitution_coefficient>0.0</restitution_coefficient>
+          <threshold>100000.0</threshold>
+        </bounce>
+        <contact>
+          <ode>
+            <soft_cfm>0.0</soft_cfm>
+            <soft_erp>0.2</soft_erp>
+            <kp>100000.0</kp>
+            <kd>1.0</kd>
+            <max_vel>100.0</max_vel>
+            <min_depth>0.001</min_depth>
+          </ode>
+        </contact>
       </gazebo>
       <gazebo reference="right_wheel_back">
-        <mu1>0.1</mu1>
-        <mu2>0.1</mu2>
-        <kp>1000000.0</kp>
-        <kd>1.0</kd>
+        <friction>
+          <ode>
+            <mu>1.01</mu>
+            <mu2>1.01</mu2>
+            <fdir1>0 0 1</fdir1>
+            <slip1>0</slip1>
+            <slip2>0</slip2>
+          </ode>
+        </friction>
+        <bounce>
+          <restitution_coefficient>0.0</restitution_coefficient>
+          <threshold>100000.0</threshold>
+        </bounce>
+        <contact>
+          <ode>
+            <soft_cfm>0.0</soft_cfm>
+            <soft_erp>0.2</soft_erp>
+            <kp>100000.0</kp>
+            <kd>1.0</kd>
+            <max_vel>100.0</max_vel>
+            <min_depth>0.001</min_depth>
+          </ode>
+        </contact>
       </gazebo>
       <!-- https://osrf-migration.github.io/sdformat-gh-pages/#!/osrf/sdformat/issues/131/page/1-->

Commit message: Create a nav config file for bigger forklift

File: src/forklift_controller/urdf/robot.urdf.xacro (robot description, xacro)
@@ -11,6 +11,6 @@
       <right_joint>right_wheel_joint</right_joint>
       <right_joint>right_wheel_back_joint</right_joint>
-      <wheel_separation>0.895</wheel_separation>
-      <wheel_radius>0.07</wheel_radius>
+      <wheel_separation>0.890</wheel_separation>
+      <wheel_radius>0.25</wheel_radius>
       <odom_publish_frequency>30</odom_publish_frequency>
       <odom_topic>$(arg namespace)/odom</odom_topic>

File: src/forklift_controller/urdf/robot_core.xacro (robot description, xacro)
@@ -124,5 +124,5 @@
     <parent link="base_link" />
     <child link="rplidar_link" />
-    <origin xyz="0 0 0.4" rpy="0 0 0" />
+    <origin xyz="0 0 1" rpy="0 0 0" />
   </joint>
   <gazebo reference="rplidar_link">
@@ -153,4 +153,5 @@
     <preserveFixedJoint>true</preserveFixedJoint>
   </gazebo>
+  <!--https://medium.com/@alitekes1/gazebo-sim-plugin-and-sensors-for-acquire-data-from-simulation-environment-681d8e2ad853-->
   <!--
   <gazebo reference="fork_plate_joint">

Commit message: Fix nav2 configuration

File: src/forklift_controller/urdf/robot.urdf.xacro (robot description, xacro)
@@ -23,5 +23,5 @@
       <max_angular_acceleration>20</max_angular_acceleration>
       <min_angular_acceleration>-20</min_angular_acceleration>
-      <max_linear_velocity>0.5</max_linear_velocity>
+      <max_linear_velocity>6</max_linear_velocity>
       <min_linear_velocity>-0.5</min_linear_velocity>
       <max_angular_velocity>10</max_angular_velocity>

File: src/forklift_controller/urdf/robot_core.xacro (robot description, xacro)
@@ -74,5 +74,5 @@
     <parent link="base_link" />
     <child link="fork_plate" />
-    <origin xyz="1.25 0 0.3" rpy="0 0 0" />
+    <origin xyz="1.25 0 0.25" rpy="0 0 0" />
     <axis xyz="0 0 1" />
     <limit effort="110" lower="-0.15" upper="0.6" velocity="0.5" />
@@ -80,8 +80,8 @@
   <xacro:fork id="1" mass="15" scale="1" fork_attach_offsets="0.05 0.2 -0.35"></xacro:fork>
   <xacro:fork id="2" mass="15" scale="1" fork_attach_offsets="0.05 -0.2 -0.35"></xacro:fork>
-  <xacro:wheel name="right_wheel" mass="5" scale="1" x="0.8" y="-0.4" z="-0.35" roll="${pi}"></xacro:wheel>
-  <xacro:wheel name="right_wheel_back" mass="5" scale="1" x="-0.65" y="-0.4" z="-0.35" roll="${pi}"></xacro:wheel>
-  <xacro:wheel name="left_wheel" mass="5" scale="1" x="0.8" y="0.4" z="-0.35" roll="${pi}"></xacro:wheel>
-  <xacro:wheel name="left_wheel_back" mass="5" scale="1" x="-0.65" y="0.4" z="-0.35" roll="${pi}"></xacro:wheel>
+  <xacro:wheel name="right_wheel" mass="5" scale="1" x="0.8" y="-0.4" z="-0.35" yaw="${pi/2}" axis="-1"></xacro:wheel>
+  <xacro:wheel name="right_wheel_back" mass="5" scale="1" x="-0.65" y="-0.4" z="-0.35" yaw="${pi/2}" axis="-1"></xacro:wheel>
+  <xacro:wheel name="left_wheel" mass="5" scale="1" x="0.8" y="0.4" z="-0.35" yaw="-${pi/2}"  axis="-1"></xacro:wheel>
+  <xacro:wheel name="left_wheel_back" mass="5" scale="1" x="-0.65" y="0.4" z="-0.35" yaw="-${pi/2}" axis="-1"></xacro:wheel>
   <gazebo>
     <!--
@@ -122,5 +122,5 @@
     <parent link="base_link" />
     <child link="rplidar_link" />
-    <origin xyz="0 0 1" rpy="0 0 0" />
+    <origin xyz="0 0 1.5" rpy="0 0 0" />
   </joint>
   <gazebo reference="rplidar_link">

File: src/forklift_controller/urdf/wheel.xacro (robot description, xacro)
@@ -4,15 +4,14 @@
     <xacro:property name="wheel_radius" value="0.25" />
     <xacro:include filename="inertial_macros.xacro" />
-    <xacro:macro name="wheel" params="name mass scale x y z roll">
+    <xacro:macro name="wheel" params="name mass scale x y z yaw axis">
   <joint name="${name}_joint" type="continuous">
     <parent link="base_link" />
     <child link="${name}" />
-    <origin xyz="${x} ${y} ${z}" rpy="-${pi/2} 0 ${roll}" />
-    <origin xyz="${x} ${y} ${z}" rpy="-${pi/2}} 0 ${roll}" />
-    <axis xyz="0 0 -1" />
+    <origin xyz="${x} ${y} ${z}" rpy="${pi/2} 0 0" />
+    <axis xyz="0 0 ${axis}" />
   </joint>
   <link name="${name}">
     <visual>
-      <origin xyz="0 0 0" rpy="-${pi/2} 0 0" />
+      <origin xyz="0 0 0" rpy="${yaw} 0 0" />
       <geometry>
         <!--The
