Commit message: Refactor and implement contact sensor

File: src/forklift_controller/urdf/robot_core.xacro (robot description, xacro)
@@ -217,3 +217,20 @@
         </xacro:inertial_cylinder>
     </link>
+    <gazebo>
+    <plugin filename="gz-sim-touchplugin-system"
+                    name="gz::sim::systems::TouchPlugin">
+                <target>cube</target>
+                <time>0.001</time>
+                <namespace>forklift</namespace>
+                <enabled>true</enabled>
+            </plugin>
+    </gazebo>
+    <gazebo reference="fork_plate">
+            <sensor name='sensor_contact' type='contact'>
+                    <contact>
+                        <collision>fork_plate_fixed_joint_lump__fork_1_collision_1</collision>
+                        <topic>forklift/container_contact</topic>
+                    </contact>
+            </sensor>
+        </gazebo>
 </robot>

Commit message: Add different LLM model choices to GUI

File: src/forklift_controller/urdf/robot_core.xacro (robot description, xacro)
@@ -20,13 +20,12 @@
     <xacro:property name="base_height" value="0.15"/>
     <xacro:property name="base_width" value="0.3"/>
-    <link name="base_footprint">
-    </link>
-    <!-- base_link LINK -->
+    <link name="base_link">
+    </link>
     <joint name="base_link_joint" type="fixed">
-        <parent link="base_footprint"/>
-        <child link="base_link"/>
+        <parent link="base_link"/>
+        <child link="chassis"/>
         <origin xyz="0 0 0.125"/>
     </joint>
-    <link name="base_link">
+    <link name="chassis">
         <visual>
             <origin xyz="0 0 0.05"/>
@@ -67,5 +66,5 @@
     </link>
     <joint name="fork_plate_joint" type="prismatic">
-        <parent link="base_link"/>
+        <parent link="chassis"/>
         <child link="fork_plate"/>
         <!--Offset the joint position by the track depth amount-->
@@ -125,5 +124,5 @@
     <!-- LEFT WHEEL LINK -->
     <joint name="left_wheel_joint" type="continuous">
-        <parent link="base_link"/>
+        <parent link="chassis"/>
         <child link="left_wheel"/>
         <origin xyz="0.23 0.13 -0.075" rpy="0 0 0" />
@@ -148,5 +147,5 @@
     </link>
     <joint name="left_wheel_back_joint" type="continuous">
-        <parent link="base_link"/>
+        <parent link="chassis"/>
         <child link="left_wheel_back"/>
         <origin xyz="-0.2 0.13 -0.075" rpy="0 0 0" />
@@ -173,5 +172,5 @@
     <!-- RIGHT WHEEL LINK -->
     <joint name="right_wheel_joint" type="continuous">
-        <parent link="base_link"/>
+        <parent link="chassis"/>
         <child link="right_wheel"/>
         <origin xyz="0.23 -0.13 -0.075" rpy="0 0 0" />
@@ -196,5 +195,5 @@
     </link>
     <joint name="right_wheel_back_joint" type="continuous">
-        <parent link="base_link"/>
+        <parent link="chassis"/>
         <child link="right_wheel_back"/>
         <origin xyz="-0.2 -0.13 -0.075" rpy="0 0 0" />

Commit message: Small refactors

File: src/forklift_controller/urdf/robot_core.xacro (robot description, xacro)
@@ -20,17 +20,16 @@
     <xacro:property name="base_height" value="0.15"/>
     <xacro:property name="base_width" value="0.3"/>
+    <link name="base_footprint">
+    </link>
+    <joint name="base_link_joint" type="fixed">
+        <parent link="base_footprint"/>
+        <child link="base_link"/>
+        <origin xyz="0 0 0.125"/>
+    </joint>
     <link name="base_link">
-    </link>
-    <joint name="base_link_joint" type="fixed">
-        <parent link="base_link"/>
-        <child link="chassis"/>
-        <origin xyz="0 0 0.125"/>
-    </joint>
-    <link name="chassis">
         <visual>
             <origin xyz="0 0 0.05"/>
             <geometry>
                 <mesh filename="$(find forklift_controller)/meshes/body.dae" scale="0.0027 0.0027 0.0027"/>
-                <!-- <box size="0.3 ${base_width} ${base_height}"/> -->
             </geometry>
         </visual>
@@ -66,5 +65,5 @@
     </link>
     <joint name="fork_plate_joint" type="prismatic">
-        <parent link="chassis"/>
+        <parent link="base_link"/>
         <child link="fork_plate"/>
         <!--Offset the joint position by the track depth amount-->
@@ -124,5 +123,5 @@
     <!-- LEFT WHEEL LINK -->
     <joint name="left_wheel_joint" type="continuous">
-        <parent link="chassis"/>
+        <parent link="base_link"/>
         <child link="left_wheel"/>
         <origin xyz="0.23 0.13 -0.075" rpy="0 0 0" />
@@ -147,5 +146,5 @@
     </link>
     <joint name="left_wheel_back_joint" type="continuous">
-        <parent link="chassis"/>
+        <parent link="base_link"/>
         <child link="left_wheel_back"/>
         <origin xyz="-0.2 0.13 -0.075" rpy="0 0 0" />
@@ -172,5 +171,5 @@
     <!-- RIGHT WHEEL LINK -->
     <joint name="right_wheel_joint" type="continuous">
-        <parent link="chassis"/>
+        <parent link="base_link"/>
         <child link="right_wheel"/>
         <origin xyz="0.23 -0.13 -0.075" rpy="0 0 0" />
@@ -195,5 +194,5 @@
     </link>
     <joint name="right_wheel_back_joint" type="continuous">
-        <parent link="chassis"/>
+        <parent link="base_link"/>
         <child link="right_wheel_back"/>
         <origin xyz="-0.2 -0.13 -0.075" rpy="0 0 0" />
@@ -233,3 +232,32 @@
             </sensor>
         </gazebo>
+    <gazebo reference="base_link">
+    <sensor name="lidar" type="gpu_lidar">
+      <!-- <gz_frame_id>fork_plate_fixed_joint_lump__fork_1_collision_1</gz_frame_id> -->
+      <topic>scan</topic>
+      <always_on>true</always_on>
+      <visualize>true</visualize>
+      <update_rate>5</update_rate>
+      <ray>
+        <scan>
+          <horizontal>
+            <samples>360</samples>
+            <resolution>1.000000</resolution>
+            <min_angle>0.000000</min_angle>
+            <max_angle>6.280000</max_angle>
+          </horizontal>
+        </scan>
+        <range>
+          <min>0.120000</min>
+          <max>1.0</max>
+          <resolution>0.015000</resolution>
+        </range>
+        <noise>
+          <type>gaussian</type>
+          <mean>0.0</mean>
+          <stddev>0.01</stddev>
+        </noise>
+      </ray>
+    </sensor>
+  </gazebo>
 </robot>

Commit message: Add nav file for testing new implementation

File: src/forklift_controller/urdf/robot_core.xacro (robot description, xacro)
@@ -23,7 +23,7 @@
     </link>
     <joint name="base_link_joint" type="fixed">
-        <parent link="base_footprint"/>
-        <child link="base_link"/>
-        <origin xyz="0 0 0.125"/>
+        <parent link="base_link"/>
+        <child link="base_footprint"/>
+        <origin xyz="0 0 0" rpy="0 0 0"/>
     </joint>
     <link name="base_link">

Commit message: Start to refactor gui-end

File: src/forklift_controller/urdf/robot_core.xacro (robot description, xacro)
@@ -76,5 +76,5 @@
         </inertial>
     </link>
-    <joint name="fork_plate_joint" type="prismatic">
+    <joint name="fork_plate_joint" type="fixed">
         <parent link="base_link"/>
         <child link="fork_plate"/>
@@ -220,4 +220,5 @@
                 <time>0.001</time>
                 <enabled>true</enabled>
+                <!--$(arg namespace)-->
                 <namespace>$(arg namespace)</namespace>
             </plugin>

Commit message: Fix and simplify pickup function

File: src/forklift_controller/urdf/robot_core.xacro (robot description, xacro)
@@ -235,23 +235,21 @@
             <origin xyz="0 0 0" rpy="0 0 0"/>
             <geometry>
-                <box size="0.01 0.1 0.2"/>
-            </geometry>
-        </visual>
-        <collision>
-            <origin xyz="0 0 0" rpy="0 0 0"/>
-            <geometry>
-                <box size="0.01 0.3 0.2"/>
-            </geometry>
-        </collision>
-        <inertial>
-            <mass value="75"/>
-            <origin xyz="0.005 0.15 0.1" rpy="0 0 0"/>
-            <inertia ixx="0.075" ixy="0" ixz="0" iyy="0.075" iyz="0" izz="0.0045"/>
-        </inertial>
+              <cylinder radius="0.03" length="0.03"></cylinder>
+            </geometry>
+        </visual>
+        <collision>
+            <origin xyz="0 0 0" rpy="0 0 0"/>
+            <geometry>
+              <cylinder radius="0.03" length="0.03"></cylinder>
+            </geometry>
+        </collision>
+       <xacro:inertial_cylinder mass="0.1" length="0.03" radius="0.03">
+            <origin xyz="0 0 0" rpy="0 0 0"/>
+        </xacro:inertial_cylinder>
     </link>
     <joint name="rplidar_joint" type="fixed">
         <parent link="base_link"/>
         <child link="rplidar_link"/>
-        <origin xyz="0 0 0.5" rpy="0 0 0"/>
+        <origin xyz="-0.23 0 0.14" rpy="0 0 0"/>
     </joint>
     <gazebo reference="rplidar_link">

Commit message: Start mergin GUI

File: src/forklift_controller/urdf/robot_core.xacro (robot description, xacro)
@@ -15,4 +15,5 @@
     </material>
     <!-- BASE LINK -->
+    <xacro:property name="scaler" value="1.0"/>
     <xacro:property name="track_length" value="0.3"/>
     <xacro:property name="track_depth" value="0.02"/> <!--This is actually the depth of the track when in up position-->
@@ -29,5 +30,5 @@
             <origin rpy="0 0 0" xyz="0 0 0"/>
             <geometry>
-              <box size="0.001 0.001 0.001"/>
+              <box size="${scaler*0.001} ${scaler*0.001} ${scaler*0.001}"/>
             </geometry>
           </visual>
@@ -36,5 +37,5 @@
         <parent link="base_link"/>
         <child link="base_footprint"/>
-        <origin xyz="0 0 -0.15" rpy="0 0 0"/>
+        <origin xyz="${scaler*0} ${scaler*0} ${scaler*-0.15}" rpy="0 0 0"/>
     </joint>
     <link name="base_link">
@@ -48,6 +49,6 @@
             <origin xyz="0 0 0"/>
             <geometry>
-                <mesh filename="$(find forklift_controller)/meshes/body.dae" scale="0.0027 0.0027 0.0027"/>
-                <!-- <box size="0.3 ${base_width} ${base_height}"/> -->
+                <mesh filename="$(find forklift_controller)/meshes/body.dae"
+                  scale="${scaler*0.0027} ${scaler*0.0027} ${scaler*0.0027}"/>
             </geometry>
         </collision>

Commit message: Implement working back and forth messaging

File: src/forklift_controller/urdf/robot_core.xacro (robot description, xacro)
@@ -252,5 +252,5 @@
         <parent link="base_link"/>
         <child link="rplidar_link"/>
-        <origin xyz="-0.23 0 0.14" rpy="0 0 0"/>
+        <origin xyz="0 0 0.4" rpy="0 0 0"/>
     </joint>
     <gazebo reference="rplidar_link">

Commit message: Refactor models folder

File: src/forklift_controller/urdf/robot_core.xacro (robot description, xacro)
@@ -43,5 +43,5 @@
             <origin xyz="0 0 0"/>
             <geometry>
-                <mesh filename="$(find forklift_controller)/meshes/body.dae" scale="0.0027 0.0027 0.0027"/>
+                <mesh filename="$(find forklift_controller)/models/forklift/meshes/body.dae" scale="0.0027 0.0027 0.0027"/>
             </geometry>
         </visual>
@@ -49,5 +49,5 @@
             <origin xyz="0 0 0"/>
             <geometry>
-                <mesh filename="$(find forklift_controller)/meshes/body.dae"
+                <mesh filename="$(find forklift_controller)/models/forklift/meshes/body.dae"
                   scale="${scaler*0.0027} ${scaler*0.0027} ${scaler*0.0027}"/>
             </geometry>
@@ -62,5 +62,5 @@
             <geometry>
                 <!-- <box size="0.01 0.2 0.2"/> -->
-                <mesh filename="$(find forklift_controller)/meshes/fork_plate.dae" scale="0.0027 0.0027 0.0027"/>
+                <mesh filename="$(find forklift_controller)/models/forklift/meshes/fork_plate.dae" scale="0.0027 0.0027 0.0027"/>
             </geometry>
         </visual>
@@ -178,5 +178,6 @@
             <origin xyz="0 0 0" rpy="-${pi/2} 0 0"/>
             <geometry>
-                <mesh filename="$(find forklift_controller)/meshes/front_wheel_right.dae" scale="0.002 0.002 0.002"/>
+              <mesh filename="package://forklift_controller/models/forklift/meshes/front_wheel_right.dae" scale="0.002 0.002 0.002"/>
+              <!-- <mesh filename="$(find forklift_controller)/meshes/front_wheel_right.dae" scale="0.002 0.002 0.002"/> -->
             </geometry>
         </visual>
@@ -202,5 +203,5 @@
             <origin xyz="0 0 0" rpy="${pi/2} 0 0"/>
             <geometry>
-                <mesh filename="$(find forklift_controller)/meshes/front_wheel_right.dae" scale="0.002 0.002 0.002"/>
+                <mesh filename="$(find forklift_controller)/models/forklift/meshes/front_wheel_right.dae" scale="0.002 0.002 0.002"/>
             </geometry>
         </visual>
@@ -292,5 +293,5 @@
             <origin xyz="0 0 0" rpy="${pi/2} 0 0"/>
             <geometry>
-                <mesh filename="$(find forklift_controller)/meshes/front_wheel_right.dae" scale="0.002 0.002 0.002"/>
+                <mesh filename="$(find forklift_controller)/models/forklift/meshes/front_wheel_right.dae" scale="0.002 0.002 0.002"/>
             </geometry>
         </visual>
@@ -315,5 +316,5 @@
             <origin xyz="0 0 0" rpy="-${pi/2} 0 0"/>
             <geometry>
-                <mesh filename="$(find forklift_controller)/meshes/front_wheel_right.dae" scale="0.002 0.002 0.002"/>
+                <mesh filename="$(find forklift_controller)/models/forklift/meshes/front_wheel_right.dae" scale="0.002 0.002 0.002"/>
             </geometry>
         </visual>

Commit message: Add new map and create slam util launch

File: src/forklift_controller/urdf/robot_core.xacro (robot description, xacro)
@@ -178,6 +178,5 @@
             <origin xyz="0 0 0" rpy="-${pi/2} 0 0"/>
             <geometry>
-              <mesh filename="package://forklift_controller/models/forklift/meshes/front_wheel_right.dae" scale="0.002 0.002 0.002"/>
-              <!-- <mesh filename="$(find forklift_controller)/meshes/front_wheel_right.dae" scale="0.002 0.002 0.002"/> -->
+              <mesh filename="$(find forklift_controller)/models/forklift/meshes/front_wheel_right.dae" scale="0.002 0.002 0.002"/>
             </geometry>
         </visual>
@@ -203,5 +202,5 @@
             <origin xyz="0 0 0" rpy="${pi/2} 0 0"/>
             <geometry>
-                <mesh filename="$(find forklift_controller)/models/forklift/meshes/front_wheel_right.dae" scale="0.002 0.002 0.002"/>
+              <mesh filename="$(find forklift_controller)/models/forklift/meshes/front_wheel_right.dae" scale="0.002 0.002 0.002"/>
             </geometry>
         </visual>

Commit message: Replace simple fork with complex shape

File: src/forklift_controller/urdf/robot_core.xacro (robot description, xacro)
@@ -87,13 +87,15 @@
     <link name="fork_1">
         <visual>
-            <origin xyz="0.15 0 0" rpy="0 0 0"/>
-            <geometry>
-                <box size="0.3 0.05 0.01"/>
-            </geometry>
-        </visual>
-        <collision>
-            <origin xyz="0.15 0 0" rpy="0 0 0"/>
-            <geometry>
-                <box size="0.3 0.05 0.01"/>
+            <origin xyz="0 0.02 0" rpy="0 0 -${pi}"/>
+            <geometry>
+                <mesh filename="$(find forklift_controller)/models/forklift/meshes/fork.dae" scale="0.0027 0.0027 0.0027"/>
+                <!-- <box size="0.3 0.05 0.01"/> -->
+            </geometry>
+        </visual>
+        <collision>
+            <origin xyz="0 0 0"  rpy="0 0 -${pi}"/>
+            <geometry>
+                <mesh filename="$(find forklift_controller)/models/forklift/meshes/fork.dae" scale="0.0027 0.0027 0.0027"/>
+                <!-- <box size="0.3 0.05 0.01"/> -->
             </geometry>
         </collision>
@@ -107,17 +109,18 @@
         <parent link="fork_plate"/>
         <child link="fork_1"/>
-        <origin xyz="0 -0.05 -0.01" rpy="0 0 0"/>
+        <origin xyz="-0.02 -0.06 -0.07" rpy="0 0 0"/>
     </joint>
     <link name="fork_2">
         <visual>
-            <origin xyz="0.15 0 0" rpy="0 0 0"/>
-            <geometry>
-                <box size="0.3 0.05 0.01"/>
-            </geometry>
-        </visual>
-        <collision>
-            <origin xyz="0.15 0 0" rpy="0 0 0"/>
-            <geometry>
-                <box size="0.3 0.05 0.01"/>
+            <!-- For some reason, the another forks origin is a bit different than fork1-->
+            <origin xyz="0 0.01 0" rpy="0 0 -${pi}"/>
+            <geometry>
+              <mesh filename="$(find forklift_controller)/models/forklift/meshes/fork.dae" scale="0.0027 0.0027 0.0027"/>
+            </geometry>
+        </visual>
+        <collision>
+            <origin xyz="0 0 0" rpy="0 0 -${pi}"/>
+            <geometry>
+              <mesh filename="$(find forklift_controller)/models/forklift/meshes/fork.dae" scale="0.0027 0.0027 0.0027"/>
             </geometry>
         </collision>
@@ -131,5 +134,5 @@
         <parent link="fork_plate"/>
         <child link="fork_2"/>
-        <origin xyz="0 0.05 -0.01" rpy="0 0 0"/>
+        <origin xyz="-0.02 0.06 -0.07" rpy="0 0 0"/>
     </joint>
      <!--Offset the joint position by the track depth amount-->
@@ -341,55 +344,13 @@
         <kd>1.0</kd>
       </gazebo>
-      <!--
-  <gazebo reference="base_link">
-    <sensor type="imu" name="imu_sensor">
-      <preserveFixedJoint>true</preserveFixedJoint>
-      <always_on>true</always_on>
-      <update_rate>30</update_rate>
-      <topic>imu</topic>
-      <imu>
-        <angular_velocity>
-          <x>
-            <noise type="gaussian">
-              <mean>0.0</mean>
-              <stddev>0.0</stddev>
-            </noise>
-          </x>
-          <y>
-            <noise type="gaussian">
-              <mean>0.0</mean>
-              <stddev>0.0</stddev>
-            </noise>
-          </y>
-          <z>
-            <noise type="gaussian">
-              <mean>0.0</mean>
-              <stddev>0.0</stddev>
-            </noise>
-          </z>
-        </angular_velocity>
-        <linear_acceleration>
-          <x>
-            <noise type="gaussian">
-              <mean>0.0</mean>
-              <stddev>0.0</stddev>
-            </noise>
-          </x>
-          <y>
-            <noise type="gaussian">
-              <mean>0.0</mean>
-              <stddev>0.0</stddev>
-            </noise>
-          </y>
-          <z>
-            <noise type="gaussian">
-              <mean>0.0</mean>
-              <stddev>0.0</stddev>
-            </noise>
-          </z>
-        </linear_acceleration>
-      </imu>
-    </sensor>
-  </gazebo>
-    -->
+      <!-- https://osrf-migration.github.io/sdformat-gh-pages/#!/osrf/sdformat/issues/131/page/1-->
+      <gazebo reference="fork_1_joint">
+        <disableFixedJointLumping>true</disableFixedJointLumping>
+      </gazebo>
+      <gazebo reference="fork_2_joint">
+        <disableFixedJointLumping>true</disableFixedJointLumping>
+      </gazebo>
+      <gazebo reference="fork_plate_joint">
+        <disableFixedJointLumping>true</disableFixedJointLumping>
+      </gazebo>
 </robot>
