Commit message: Refactor forklift with inertia

File: src/forklift_controller/urdf/robot_core.xacro (robot description, xacro)
@@ -2,15 +2,7 @@
 <robot xmlns:xacro="http://www.ros.org/wiki/xacro" >
     <xacro:include filename="inertial_macros.xacro"/>
+    <xacro:include filename="fork.xacro"/>
     <material name="white">
         <color rgba="1 1 1 1" />
-    </material>
-    <material name="orange">
-        <color rgba="1 0.3 0.1 1"/>
-    </material>
-    <material name="blue">
-        <color rgba="0.2 0.2 1 1"/>
-    </material>
-    <material name="black">
-        <color rgba="0 0 0 1"/>
     </material>
     <!-- BASE LINK -->
@@ -21,13 +13,9 @@
     <xacro:property name="base_height" value="0.52"/>
     <xacro:property name="base_width" value="0.3"/>
-    <xacro:property name="base_length" value="0.68"/>
+    <xacro:property name="base_length" value="0.66"/>
+    <material name="darkgray">
+      <color rgba="0.01 0.01 0.01 1"/>
+    </material>
     <xacro:property name="fork_mass" value="15"/>
-    <!--Simple collision calculation, used for inertia-->
-    <!--
-      <origin xyz="0.042 0 0.14"/>
-            <geometry>
-              <box size="${base_length} ${base_width} ${base_height}"/>
-            </geometry>
-    -->
     <link name="base_footprint">
         <inertial>
@@ -52,15 +40,15 @@
             <origin xyz="0 0 0"/>
             <geometry>
+                <mesh filename="package://forklift_controller/models/forklift/meshes/body.dae" scale="0.0027 0.0027 0.0027"/>
+                 <!--
                 <mesh filename="$(find forklift_controller)/models/forklift/meshes/body.dae" scale="0.0027 0.0027 0.0027"/>
-            </geometry>
-        </visual>
-        <collision>
-            <origin xyz="0.042 0 0.14"/>
-            <geometry>
-              <!--
+               -->
+            </geometry>
+        </visual>
+        <collision>
+            <geometry>
                 <mesh filename="$(find forklift_controller)/models/forklift/meshes/body.dae"
                   scale="${scaler*0.0027} ${scaler*0.0027} ${scaler*0.0027}"/>
-                -->
-              <box size="${base_length} ${base_width} ${base_height}"/>
+                <!-- <mesh filename="package://forklift_controller/models/forklift/meshes/body.dae" scale="0.0027 0.0027 0.0027"/> -->
             </geometry>
         </collision>
@@ -73,5 +61,6 @@
             <origin xyz="0 0 0" rpy="0 0 0"/>
             <geometry>
-                <mesh filename="$(find forklift_controller)/models/forklift/meshes/fork_plate.dae" scale="0.0027 0.0027 0.0027"/>
+               <mesh filename="package://forklift_controller/models/forklift/meshes/fork_plate.dae" scale="0.0027 0.0027 0.0027"/>
+               <!--<mesh filename="$(find forklift_controller)/models/forklift/meshes/fork_plate.dae" scale="0.0027 0.0027 0.0027"/> -->
             </geometry>
         </visual>
@@ -86,69 +75,14 @@
         </xacro:inertial_box>
     </link>
-    <joint name="fork_plate_joint" type="fixed">
+    <joint name="fork_plate_joint" type="prismatic">
         <parent link="base_link"/>
         <child link="fork_plate"/>
-        <origin xyz="0.375 0 0.05" rpy="0 0 0"/>
+        <origin xyz="0.375 0 -0.02" rpy="0 0 0"/>
         <axis xyz="0 0 1"/>
         <limit effort="110" lower="0" upper="0.6" velocity="0.5"/>
     </joint>
-    <link name="fork_1">
-      <visual>
-          <origin xyz="0 0 0" rpy="0 0 -${pi}"/>
-          <geometry>
-              <mesh filename="$(find forklift_controller)/models/forklift/meshes/fork.dae" scale="0.0027 0.0027 0.0027"/>
-          </geometry>
-      </visual>
-      <collision>
-          <origin xyz="0 0 0"  rpy="0 0 -${pi}"/>
-          <geometry>
-              <mesh filename="$(find forklift_controller)/models/forklift/meshes/fork.dae" scale="0.0027 0.0027 0.0027"/>
-          </geometry>
-      </collision>
-      <inertial>
-          <origin xyz="-0.03808040868302371, 0.00482172099079702, -0.016262899934648207"></origin>
-          <mass value="${fork_mass}"/>
-          <inertia
-          ixx="${2.55322 * fork_mass * (0.0027**5)}"
-          ixy="${2.05649 * fork_mass * (0.0027**5)}"
-          ixz="${-2.66481 * fork_mass * (0.0027**5)}"
-          iyy="${11.5514 * fork_mass * (0.0027**5)}"
-          iyz="${1.45586  * fork_mass * (0.0027**5)}"
-          izz="${9.14891 * fork_mass * (0.0027**5)}" />
-      </inertial>
-  </link>
-    <joint name="fork_1_joint" type="fixed">
-        <parent link="fork_plate"/>
-        <child link="fork_1"/>
-        <origin xyz="-0.02 -0.06 -0.07" rpy="0 0 0"/>
-    </joint>
-    <!--
-    <link name="fork_2">
-        <visual>
-            <origin xyz="0 0 0" rpy="0 0 -${pi}"/>
-            <geometry>
-              <mesh filename="$(find forklift_controller)/models/forklift/meshes/fork.dae" scale="0.0027 0.0027 0.0027"/>
-            </geometry>
-        </visual>
-        <collision>
-            <origin xyz="0 0 0" rpy="0 0 -${pi}"/>
-            <geometry>
-              <mesh filename="$(find forklift_controller)/models/forklift/meshes/fork.dae" scale="0.0027 0.0027 0.0027"/>
-            </geometry>
-        </collision>
-        <inertial>
-            <mass value="${fork_mass}"/>
-            <inertia
-            ixx="${1.27661 * fork_mass}" ixy="${1.028245 * fork_mass}" ixz="${-1.332405 * fork_mass}"
-            iyy="${5.7757 * fork_mass}" iyz="${0.72793 * fork_mass}"
-            izz="${4.574455 * fork_mass}" />
-        </inertial>
-    </link>
-    <joint name="fork_2_joint" type="fixed">
-        <parent link="fork_plate"/>
-        <child link="fork_2"/>
-        <origin xyz="-0.02 0.06 -0.07" rpy="0 0 0"/>
-    </joint>
-    -->
+    <xacro:fork id="1" mass="15" scale="1" fork_attach_offsets="0.01 -0.05 -0.03">
+    </xacro:fork>
+    <xacro:fork id="2" mass="15" scale="1" fork_attach_offsets="0.01 0.05 -0.03"></xacro:fork>
      <!--Offset the joint position by the track depth amount-->
     <!--
@@ -189,5 +123,5 @@
         <parent link="base_link"/>
         <child link="left_wheel"/>
-        <origin xyz="0.23 0.13 -0.1" rpy="-${pi/2} 0 0" />
+        <origin xyz="0.25 0.13 -0.1" rpy="-${pi/2} 0 0" />
         <axis xyz="0 0 1"/>
     </joint>
@@ -196,5 +130,6 @@
             <origin xyz="0 0 0" rpy="-${pi/2} 0 0"/>
             <geometry>
-              <mesh filename="$(find forklift_controller)/models/forklift/meshes/front_wheel_right.dae" scale="0.002 0.002 0.002"/>
+               <mesh filename="package://forklift_controller/models/forklift/meshes/front_wheel_right.dae" scale="0.0025 0.0025 0.0025"/>
+               <!-- <mesh filename="$(find forklift_controller)/models/forklift/meshes/front_wheel_right.dae" scale="0.002 0.002 0.002"/> -->
             </geometry>
         </visual>
@@ -213,5 +148,5 @@
         <parent link="base_link"/>
         <child link="right_wheel"/>
-        <origin xyz="0.23 -0.13 -0.1" rpy="-${pi/2} 0 0" />
+        <origin xyz="0.25 -0.13 -0.1" rpy="-${pi/2} 0 0" />
         <axis xyz="0 0 1"/>
     </joint>
@@ -220,5 +155,7 @@
             <origin xyz="0 0 0" rpy="${pi/2} 0 0"/>
             <geometry>
-              <mesh filename="$(find forklift_controller)/models/forklift/meshes/front_wheel_right.dae" scale="0.002 0.002 0.002"/>
+              <!-- package://forklift_controller resolves to install/forklift_controller/share/forklift_controller-->
+              <mesh filename="package://forklift_controller/models/forklift/meshes/front_wheel_right.dae" scale="0.0025 0.0025 0.0025"/>
+              <!--<mesh filename="$(find forklift_controller)/models/forklift/meshes/front_wheel_right.dae" scale="0.002 0.002 0.002"/>  -->
             </geometry>
         </visual>
@@ -240,5 +177,5 @@
                 <enabled>true</enabled>
                 <!--$(arg namespace)-->
-                <namespace>$(arg namespace)</namespace>
+                <!-- <namespace>$(arg namespace)</namespace> -->
             </plugin>
     </gazebo>
@@ -278,5 +215,5 @@
           <always_on>true</always_on>
           <gz_frame_id>rplidar_link</gz_frame_id>
-          <topic>$(arg namespace)/scan</topic>
+          <!-- <topic>$(arg namespace)/scan</topic> -->
           <lidar>
             <scan>
@@ -310,6 +247,9 @@
             <origin xyz="0 0 0" rpy="${pi/2} 0 0"/>
             <geometry>
+                <mesh filename="package://forklift_controller/models/forklift/meshes/front_wheel_right.dae" scale="0.0025 0.0025 0.0025"/>
+                <!--
                 <mesh filename="$(find forklift_controller)/models/forklift/meshes/front_wheel_right.dae" scale="0.002 0.002 0.002"/>
-            </geometry>
+                -->
+                </geometry>
         </visual>
         <collision>
@@ -333,5 +273,8 @@
             <origin xyz="0 0 0" rpy="-${pi/2} 0 0"/>
             <geometry>
+                <mesh filename="package://forklift_controller/models/forklift/meshes/front_wheel_right.dae" scale="0.0025 0.0025 0.0025"/>
+                  <!--
                 <mesh filename="$(find forklift_controller)/models/forklift/meshes/front_wheel_right.dae" scale="0.002 0.002 0.002"/>
+                 -->
             </geometry>
         </visual>
@@ -447,11 +390,4 @@
         </contact>
       </gazebo>
-      <!-- https://osrf-migration.github.io/sdformat-gh-pages/#!/osrf/sdformat/issues/131/page/1-->
-      <gazebo reference="fork_1_joint">
-        <disableFixedJointLumping>true</disableFixedJointLumping>
-      </gazebo>
-      <gazebo reference="fork_2_joint">
-        <disableFixedJointLumping>true</disableFixedJointLumping>
-      </gazebo>
       <gazebo reference="fork_plate_joint">
         <disableFixedJointLumping>true</disableFixedJointLumping>

File: src/forklift_controller/urdf/test.urdf (robot description, URDF)
Before this commit: robot forklift, 9 links, 8 joints
Links:
- added link fork_1_attach, mass 7.5; collision box size=0.15 0.025 0.01; visual box size=0.15 0.025 0.01
- added link fork_2, mass 7.5; collision box size=0.2 0.025 0.005; visual box size=0.2 0.025 0.005
- added link fork_2_attach, mass 7.5; collision box size=0.15 0.025 0.01; visual box size=0.15 0.025 0.01
- link base_link: geometry collision mesh filename=/home/elmeripk/forklift_sim/install/forklift_controller/sha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 scale=0.0027 0.0027 0.0027; visual mesh filename=/home/elmeripk/forklift_sim/install/forklift_controller/sha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 scale=0.0027 0.0027 0.0027
- link fork_1: mass None -> 7.5; geometry collision box size=0.2 0.025 0.005; visual box size=0.2 0.025 0.005
Joints:
- added joint fork_2_joint: type fixed, parent fork_2_attach, child fork_2, origin xyz=0.005 0 -0.11249999999999999 rpy=0 0 0
- added joint fork_attach_1_joint: type fixed, parent fork_plate, child fork_1_attach, origin xyz=0.01 -0.05 -0.03 rpy=0 0 0
- added joint fork_attach_2_joint: type fixed, parent fork_plate, child fork_2_attach, origin xyz=0.01 0.05 -0.03 rpy=0 0 0
- joint fork_1_joint: origin xyz=-0.02 -0.06 -0.07 rpy=0 0 0 -> xyz=0.005 0 -0.11249999999999999 rpy=0 0 0; parent fork_plate -> fork_1_attach
- joint fork_plate_joint: origin xyz=0.375 0 0.05 rpy=0 0 0 -> xyz=0.375 0 -0.02 rpy=0 0 0; type fixed -> prismatic
- joint left_wheel_joint: origin xyz=0.23 0.13 -0.1 rpy=-1.5707963267948966 0 0 -> xyz=0.25 0.13 -0.1 rpy=-1.5707963267948966 0 0
- joint right_wheel_joint: origin xyz=0.23 -0.13 -0.1 rpy=-1.5707963267948966 0 0 -> xyz=0.25 -0.13 -0.1 rpy=-1.5707963267948966 0 0

Commit message: Fix issue with smac planner

File: src/forklift_controller/urdf/robot_core.xacro (robot description, xacro)
@@ -16,16 +16,16 @@
   </material>
   <xacro:property name="fork_mass" value="15" />
+  <!--See: https://github.com/ros-navigation/navigation2_tutorials/blob/rolling/sam_bot_description/src/description/sam_bot_description.urdf -->
+  <!--From nav2 docs:
+  "We will also be using the box_inertia macro we defined before to add some inertial properties
+  to our base_link. The kdl_parser package used in robot_state_publisher
+  doesn’t like inertial properties being specified in the root link,
+  in this case the base_link, to combat this we will be including them in the base_footprint instead.
+  Include the following code snippet within <link name="base_footprint"> tag of base_footprint in our URDF."
+  -->
   <link name="base_footprint">
-    <inertial>
-      <mass value="0.0001" />
-      <origin xyz="0 0 0" />
-      <inertia ixx="0.0001" ixy="0.0" ixz="0.0" iyy="0.0001" iyz="0.0" izz="0.0001" />
-    </inertial>
-    <visual>
-      <origin rpy="0 0 0" xyz="0 0 0" />
-      <geometry>
-        <box size="0.001 0.001 0.001" />
-      </geometry>
-    </visual>
+    <xacro:inertial_box mass="50" x="${base_length}" y="${base_width}" z="${base_height}">
+      <origin xyz="-0.1 0 ${0.35+0.25}" rpy="0 0 0" />
+    </xacro:inertial_box>
   </link>
   <joint name="base_link_joint" type="fixed">
@@ -43,11 +43,9 @@
     </visual>
     <collision>
+      <origin xyz="0 0 0" />
       <geometry>
         <mesh filename="package://forklift_controller/models/forklift/meshes/body_correct_scale.dae"/>
       </geometry>
     </collision>
-    <xacro:inertial_box mass="50" x="${base_length}" y="${base_width}" z="${base_height}">
-      <origin xyz="-0.1 0 0" rpy="0 0 0" />
-    </xacro:inertial_box>
   </link>
   <xacro:property name="plate_width" value="0.885"/>
@@ -82,6 +80,6 @@
   <xacro:fork id="1" mass="15" scale="1" fork_attach_offsets="0.05 0.2 -0.35"></xacro:fork>
   <xacro:fork id="2" mass="15" scale="1" fork_attach_offsets="0.05 -0.2 -0.35"></xacro:fork>
-  <xacro:wheel name="right_wheel" mass="5" scale="1" x="0.8" y="-0.4" z="-0.35" roll="0"></xacro:wheel>
-  <xacro:wheel name="right_wheel_back" mass="5" scale="1" x="-0.65" y="-0.4" z="-0.35" roll="0"></xacro:wheel>
+  <xacro:wheel name="right_wheel" mass="5" scale="1" x="0.8" y="-0.4" z="-0.35" roll="${pi}"></xacro:wheel>
+  <xacro:wheel name="right_wheel_back" mass="5" scale="1" x="-0.65" y="-0.4" z="-0.35" roll="${pi}"></xacro:wheel>
   <xacro:wheel name="left_wheel" mass="5" scale="1" x="0.8" y="0.4" z="-0.35" roll="${pi}"></xacro:wheel>
   <xacro:wheel name="left_wheel_back" mass="5" scale="1" x="-0.65" y="0.4" z="-0.35" roll="${pi}"></xacro:wheel>

File: src/forklift_controller/urdf/wheel.xacro (robot description, xacro)
@@ -10,5 +10,5 @@
     <origin xyz="${x} ${y} ${z}" rpy="-${pi/2} 0 ${roll}" />
     <origin xyz="${x} ${y} ${z}" rpy="-${pi/2}} 0 ${roll}" />
-    <axis xyz="0 0 1" />
+    <axis xyz="0 0 -1" />
   </joint>
   <link name="${name}">

Commit message: Fix model path

File: src/forklift_controller/urdf/robot_core.xacro (robot description, xacro)
@@ -74,5 +74,5 @@
     <parent link="base_link" />
     <child link="fork_plate" />
-    <origin xyz="1.25 0 0.25" rpy="0 0 0" />
+    <origin xyz="1.25 0 0.09" rpy="0 0 0" />
     <axis xyz="0 0 1" />
     <limit effort="110" lower="-0.15" upper="0.6" velocity="0.5" />
