Commit message: Fix joint efforts for forks

File: src/forklift_controller/urdf/robot.urdf (robot description, URDF)
Before this commit: robot forklift, 12 links, 11 joints
Links:
- link base_footprint: mass 50 -> 1500
Joints:
- joint fork_plate_joint: limit lower=-0.15 upper=0.6 effort=110 velocity=0.5 -> lower=0.0 upper=5.0 effort=2500 velocity=0.5; origin xyz=1.25 0 0.3 rpy=0 0 0 -> xyz=1.15 0 0.09 rpy=0 0 0

File: src/forklift_controller/urdf/robot.urdf.xacro (robot description, xacro)
@@ -43,12 +43,17 @@
       <topic>$(arg namespace)/joint_states</topic>
     </plugin>
-    <!--
       <plugin filename="gz-sim-joint-position-controller-system"
     name="gz::sim::systems::JointPositionController">
         <joint_name>fork_plate_joint</joint_name>
-        <topic>fork_control</topic>
-        <initial_position>0.6</initial_position>
+        <initial_position>0.0</initial_position>
+        <topic>$(arg namespace)/fork_control</topic>
+        <p_gain>4000000</p_gain>
+        <i_gain>2000</i_gain>
+        <d_gain>5000</d_gain>
+        <i_min>-2000</i_min>
+        <i_max>2000</i_max>
+        <cmd_min>-80000</cmd_min>
+        <cmd_max>120000</cmd_max>
       </plugin>
-      -->
   </gazebo>
 </robot>

File: src/forklift_controller/urdf/robot_core.xacro (robot description, xacro)
@@ -25,5 +25,5 @@
   -->
   <link name="base_footprint">
-    <xacro:inertial_box mass="50" x="${base_length}" y="${base_width}" z="${base_height}">
+    <xacro:inertial_box mass="1500" x="${base_length}" y="${base_width}" z="${base_height}">
       <origin xyz="-0.1 0 ${0.35+0.25}" rpy="0 0 0" />
     </xacro:inertial_box>
@@ -74,7 +74,7 @@
     <parent link="base_link" />
     <child link="fork_plate" />
-    <origin xyz="1.25 0 0.09" rpy="0 0 0" />
+    <origin xyz="1.15 0 0.09" rpy="0 0 0" />
     <axis xyz="0 0 1" />
-    <limit effort="110" lower="-0.15" upper="0.6" velocity="0.5" />
+    <limit effort="2500" lower="0.0" upper="5.0" velocity="0.5" />
   </joint>
   <xacro:fork id="1" mass="15" scale="1" fork_attach_offsets="0.05 0.2 -0.35"></xacro:fork>
