Commit message: Refactor forklift launch to match drone

File: src/forklift_cpp/urdf/robot.urdf.xacro (robot description, xacro)
@@ -4,4 +4,13 @@
   <xacro:include filename="robot_core.xacro" />
   <gazebo>
+    <!-- <plugin
+      filename="gz-sim-pose-publisher-system"
+      name="gz::sim::systems::PosePublisher">
+      <publish_link_pose>true</publish_link_pose>
+      <publish_collision_pose>false</publish_collision_pose>
+      <publish_visual_pose>false</publish_visual_pose>
+      <publish_nested_model_pose>false</publish_nested_model_pose>
+      <use_pose_vector_msg>true</use_pose_vector_msg>
+    </plugin> -->
     <plugin
       filename="gz-sim-diff-drive-system"
@@ -41,5 +50,5 @@
       <joint_name>fork_plate</joint_name>
       -->
-      <joint_name>fork_plate</joint_name>
+      <!-- <joint_name>fork_plate</joint_name> -->
       <topic>$(arg namespace)/joint_states</topic>
     </plugin>

File: src/forklift_cpp/urdf/robot_core.xacro (robot description, xacro)
@@ -41,5 +41,5 @@
       <origin xyz="0 0 0" />
       <geometry>
-        <mesh filename="package://forklift_controller/models/forklift/meshes/body_correct_scale.dae"/>
+        <mesh filename="package://forklift_cpp/models/forklift/meshes/body_correct_scale.dae"/>
       </geometry>
     </visual>
@@ -47,5 +47,5 @@
       <origin xyz="0 0 0" />
       <geometry>
-        <mesh filename="package://forklift_controller/models/forklift/meshes/body_correct_scale.dae"/>
+        <mesh filename="package://forklift_cpp/models/forklift/meshes/body_correct_scale.dae"/>
       </geometry>
     </collision>
@@ -58,5 +58,5 @@
       <origin xyz="0 0 0" rpy="0 0 0" />
       <geometry>
-        <mesh filename="package://forklift_controller/models/forklift/meshes/fork_plate_correct_scale.dae"
+        <mesh filename="package://forklift_cpp/models/forklift/meshes/fork_plate_correct_scale.dae"
         scale="1 1 0.77"
         />

File: src/forklift_cpp/urdf/wheel.xacro (robot description, xacro)
@@ -16,6 +16,6 @@
       <geometry>
         <!--The
-        package resolves into install/forklift_controller/share/forklift_controller/-->
-        <mesh filename="package://forklift_controller/models/forklift/meshes/wheel_correct_scale.dae"/>
+        package resolves into install/forklift_cpp/share/forklift_cpp/-->
+        <mesh filename="package://forklift_cpp/models/forklift/meshes/wheel_correct_scale.dae"/>
       </geometry>
     </visual>
