Commit message: Add more licensing

File: src/forklift_cpp/urdf/inertial_macros.xacro (robot description, xacro)
@@ -1,37 +1,33 @@
 <?xml version="1.0"?>
-    <!--
-        Copyright (c) Elmeri Pohjois-Koivisto
-        See robot.urdf.xacro for licensing
-    -->
 <robot xmlns:xacro="http://www.ros.org/wiki/xacro">
-    <!-- Specify some standard inertial calculations
+  <!-- Specify some standard inertial calculations
     https://en.wikipedia.org/wiki/List_of_moments_of_inertia -->
-    <!-- These make use of xacro's mathematical functionality -->
-    <xacro:macro name="inertial_sphere" params="mass radius *origin">
-        <inertial>
-            <xacro:insert_block name="origin" />
-            <mass value="${mass}" />
-            <inertia ixx="${(2/5) * mass * (radius*radius)}" ixy="0.0" ixz="0.0"
-                iyy="${(2/5) * mass * (radius*radius)}" iyz="0.0"
-                izz="${(2/5) * mass * (radius*radius)}" />
-        </inertial>
-    </xacro:macro>
-    <xacro:macro name="inertial_box" params="mass x y z *origin">
-        <inertial>
-            <xacro:insert_block name="origin" />
-            <mass value="${mass}" />
-            <inertia ixx="${(1/12) * mass * (y*y+z*z)}" ixy="0.0" ixz="0.0"
-                iyy="${(1/12) * mass * (x*x+z*z)}" iyz="0.0"
-                izz="${(1/12) * mass * (x*x+y*y)}" />
-        </inertial>
-    </xacro:macro>
-    <xacro:macro name="inertial_cylinder" params="mass length radius *origin">
-        <inertial>
-            <xacro:insert_block name="origin" />
-            <mass value="${mass}" />
-            <inertia ixx="${(1/12) * mass * (3*radius*radius + length*length)}" ixy="0.0" ixz="0.0"
-                iyy="${(1/12) * mass * (3*radius*radius + length*length)}" iyz="0.0"
-                izz="${(1/2) * mass * (radius*radius)}" />
-        </inertial>
-    </xacro:macro>
+  <!-- These make use of xacro's mathematical functionality -->
+  <xacro:macro name="inertial_sphere" params="mass radius *origin">
+    <inertial>
+      <xacro:insert_block name="origin" />
+      <mass value="${mass}" />
+      <inertia ixx="${(2/5) * mass * (radius*radius)}" ixy="0.0" ixz="0.0"
+        iyy="${(2/5) * mass * (radius*radius)}" iyz="0.0"
+        izz="${(2/5) * mass * (radius*radius)}" />
+    </inertial>
+  </xacro:macro>
+  <xacro:macro name="inertial_box" params="mass x y z *origin">
+    <inertial>
+      <xacro:insert_block name="origin" />
+      <mass value="${mass}" />
+      <inertia ixx="${(1/12) * mass * (y*y+z*z)}" ixy="0.0" ixz="0.0"
+        iyy="${(1/12) * mass * (x*x+z*z)}" iyz="0.0"
+        izz="${(1/12) * mass * (x*x+y*y)}" />
+    </inertial>
+  </xacro:macro>
+  <xacro:macro name="inertial_cylinder" params="mass length radius *origin">
+    <inertial>
+      <xacro:insert_block name="origin" />
+      <mass value="${mass}" />
+      <inertia ixx="${(1/12) * mass * (3*radius*radius + length*length)}" ixy="0.0" ixz="0.0"
+        iyy="${(1/12) * mass * (3*radius*radius + length*length)}" iyz="0.0"
+        izz="${(1/2) * mass * (radius*radius)}" />
+    </inertial>
+  </xacro:macro>
 </robot>

File: src/forklift_cpp/urdf/robot.urdf.xacro (robot description, xacro)
@@ -1,15 +1,3 @@
 <?xml version="1.0"?>
-  <!--
-    Copyright (c) Elmeri Pohjois-Koivisto
-    Licensed under MIT license (code) and CC-BY-4.0 (models and textures),
-    see LICENSES at the repository root for full license(s)
-    Model information:
-      Model name: Forklift low poly
-      Original author: Ricardo Sanchez (https://sketchfab.com/380660711785)
-      Original URL: https://sketchfab.com/3d-models/forklift-low-poly-8ab650b3982243f8b661142de50f79c9
-    Changes made:
-      - Extracted forks, wheels and the body to a separate dae models
-      - Resized wheels, forks and the body to match proportions in meshes/models_src/forklift_spec.pdf
-  -->
 <robot xmlns:xacro="http://www.ros.org/wiki/xacro" name="forklift">
   <xacro:arg name="namespace" default="" />
@@ -65,17 +53,17 @@
       <topic>$(arg namespace)/joint_states</topic>
     </plugin>
-      <plugin filename="gz-sim-joint-position-controller-system"
-    name="gz::sim::systems::JointPositionController">
-        <joint_name>fork_plate_joint</joint_name>
-        <initial_position>0.0</initial_position>
-        <topic>$(arg namespace)/fork_control</topic>
-        <p_gain>4000000</p_gain>
-        <i_gain>2000</i_gain>
-        <d_gain>5000</d_gain>
-        <i_min>-2000</i_min>
-        <i_max>2000</i_max>
-        <cmd_min>-80000</cmd_min>
-        <cmd_max>120000</cmd_max>
-      </plugin>
+    <plugin filename="gz-sim-joint-position-controller-system"
+      name="gz::sim::systems::JointPositionController">
+      <joint_name>fork_plate_joint</joint_name>
+      <initial_position>0.0</initial_position>
+      <topic>$(arg namespace)/fork_control</topic>
+      <p_gain>4000000</p_gain>
+      <i_gain>2000</i_gain>
+      <d_gain>5000</d_gain>
+      <i_min>-2000</i_min>
+      <i_max>2000</i_max>
+      <cmd_min>-80000</cmd_min>
+      <cmd_max>120000</cmd_max>
+    </plugin>
   </gazebo>
 </robot>

File: src/forklift_cpp/urdf/robot_core.xacro (robot description, xacro)
@@ -1,7 +1,3 @@
 <?xml version="1.0"?>
-  <!--
-    Copyright (c) Elmeri Pohjois-Koivisto
-    See robot.urdf.xacro for licensing
-  -->
 <robot xmlns:xacro="http://www.ros.org/wiki/xacro">
   <xacro:include filename="inertial_macros.xacro" />

File: src/forklift_cpp/urdf/wheel.xacro (robot description, xacro)
@@ -1,7 +1,3 @@
 <?xml version="1.0" encoding="UTF-8"?>
-<!--
-  Copyright (c) Elmeri Pohjois-Koivisto
-  See robot.urdf.xacro for licensing
--->
 <robot xmlns:xacro="http://www.ros.org/wiki/xacro">
   <xacro:property name="wheel_width" value="0.15" />
