Commit message: Texture changes

File: src/forklift_cpp/urdf/robot_core.xacro (robot description, xacro)
@@ -58,5 +58,6 @@
   </link>
   <xacro:property name="plate_width" value="0.885" />
-  <xacro:property name="plate_height" value="1.290" />
+  <!-- <xacro:property name="plate_height" value="1.290" /> -->
+  <xacro:property name="plate_height" value="0.95" />
   <xacro:property name="plate_length" value="0.1" />
   <link name="fork_plate">
@@ -70,5 +71,6 @@
     </visual>
     <collision>
-      <origin xyz="0 0 0" rpy="0 0 0" />
+      <!--Move the collision down a small amount because the shape is not exactly the same size as the mesh-->
+      <origin xyz="0 0 -0.05" rpy="0 0 0" />
       <geometry>
         <box size="${plate_length} ${plate_width} ${plate_height}" />
@@ -82,5 +84,5 @@
     <parent link="base_link" />
     <child link="fork_plate" />
-    <origin xyz="1.15 0 0.09" rpy="0 0 0" />
+    <origin xyz="1.15 0 0.025" rpy="0 0 0" />
     <axis xyz="0 0 1" />
     <limit effort="2500" lower="0.0" upper="5.0" velocity="0.5" />
