Commit message: Add licenses to forklift urdf

File: src/forklift_cpp/urdf/fork.xacro (robot description, xacro)
@@ -1,3 +1,7 @@
 <?xml version="1.0"?>
+<!--
+  Copyright (c) Elmeri Pohjois-Koivisto
+  See robot.urdf.xacro for licensing
+-->
 <robot xmlns:xacro="http://www.ros.org/wiki/xacro">
   <xacro:macro name="fork" params="id mass scale fork_attach_offsets">
@@ -64,12 +68,4 @@
     </joint>
     <!-- https://osrf-migration.github.io/sdformat-gh-pages/#!/osrf/sdformat/issues/131/page/1-->
-    <!--
-    <gazebo reference="fork_{id}_joint">
-        <disableFixedJointLumping>true</disableFixedJointLumping>
-    </gazebo>
-    <gazebo reference="fork_attach_${id}_joint">
-        <disableFixedJointLumping>true</disableFixedJointLumping>
-    </gazebo>
-    -->
   </xacro:macro>
 </robot>

File: src/forklift_cpp/urdf/inertial_macros.xacro (robot description, xacro)
@@ -1,3 +1,7 @@
 <?xml version="1.0"?>
+    <!--
+        Copyright (c) Elmeri Pohjois-Koivisto
+        See robot.urdf.xacro for licensing
+    -->
 <robot xmlns:xacro="http://www.ros.org/wiki/xacro">
     <!-- Specify some standard inertial calculations

File: src/forklift_cpp/urdf/robot.urdf.xacro (robot description, xacro)
@@ -1,3 +1,15 @@
 <?xml version="1.0"?>
+  <!--
+    Copyright (c) Elmeri Pohjois-Koivisto
+    Licensed under MIT license (code) and CC-BY-4.0 (models and textures),
+    see LICENSES at the repository root for full license(s)
+    Model information:
+      Model name: Forklift low poly
+      Original author: Ricardo Sanchez (https://sketchfab.com/380660711785)
+      Original URL: https://sketchfab.com/3d-models/forklift-low-poly-8ab650b3982243f8b661142de50f79c9
+    Changes made:
+      - Extracted forks, wheels and the body to a separate dae models
+      - Resized wheels, forks and the body to match proportions in meshes/models_src/forklift_spec.pdf
+  -->
 <robot xmlns:xacro="http://www.ros.org/wiki/xacro" name="forklift">
   <xacro:arg name="namespace" default="" />

File: src/forklift_cpp/urdf/robot_core.xacro (robot description, xacro)
@@ -1,7 +1,11 @@
 <?xml version="1.0"?>
+  <!--
+    Copyright (c) Elmeri Pohjois-Koivisto
+    See robot.urdf.xacro for licensing
+  -->
 <robot xmlns:xacro="http://www.ros.org/wiki/xacro">
   <xacro:include filename="inertial_macros.xacro" />
   <xacro:include filename="fork.xacro" />
-  <xacro:include filename="wheel.xacro"/>
+  <xacro:include filename="wheel.xacro" />
   <material name="white">
     <color rgba="1 1 1 1" />
@@ -16,14 +20,18 @@
   </material>
   <xacro:property name="fork_mass" value="15" />
-  <!--See: https://github.com/ros-navigation/navigation2_tutorials/blob/rolling/sam_bot_description/src/description/sam_bot_description.urdf -->
-  <!--From nav2 docs:
+  <!--See:
+  https://github.com/ros-navigation/navigation2_tutorials/blob/rolling/sam_bot_description/src/description/sam_bot_description.urdf -->
+  <!--From
+  nav2 docs:
   "We will also be using the box_inertia macro we defined before to add some inertial properties
   to our base_link. The kdl_parser package used in robot_state_publisher
   doesn’t like inertial properties being specified in the root link,
   in this case the base_link, to combat this we will be including them in the base_footprint instead.
-  Include the following code snippet within <link name="base_footprint"> tag of base_footprint in our URDF."
+  Include the following code snippet within <link name="base_footprint"> tag of base_footprint in our
+  URDF."
   -->
   <link name="base_footprint">
-    <!--MASS HERE IS TOTALLY INACCURATE BUT WITH THE REAL MASS OF 1500, ROBOT WAS UNABLE TO TURN,
+    <!--MASS
+    HERE IS TOTALLY INACCURATE BUT WITH THE REAL MASS OF 1500, ROBOT WAS UNABLE TO TURN,
     SHOULD BE TUNED IN BOTH NAV2 AND GZ SIM DIFF DRIVE IN THE FUTURE-->
     <xacro:inertial_box mass="50" x="${base_length}" y="${base_width}" z="${base_height}">
@@ -34,5 +42,7 @@
     <parent link="base_link" />
     <child link="base_footprint" />
-    <!--Set the base_footprint down to wheel axis level + half the wheel radius to be exactly at the bottom-->
+    <!--Set
+    the base_footprint down to wheel axis level + half the wheel radius to be exactly at the
+    bottom-->
     <origin xyz="0 0 -${0.35+0.25}" rpy="0 0 0" />
   </joint>
@@ -41,5 +51,5 @@
       <origin xyz="0 0 0" />
       <geometry>
-        <mesh filename="package://forklift_cpp/models/forklift/meshes/body_correct_scale.dae"/>
+        <mesh filename="package://forklift_cpp/models/forklift/meshes/body_correct_scale.dae" />
       </geometry>
     </visual>
@@ -47,11 +57,11 @@
       <origin xyz="0 0 0" />
       <geometry>
-        <mesh filename="package://forklift_cpp/models/forklift/meshes/body_correct_scale.dae"/>
+        <mesh filename="package://forklift_cpp/models/forklift/meshes/body_correct_scale.dae" />
       </geometry>
     </collision>
   </link>
-  <xacro:property name="plate_width" value="0.885"/>
-  <xacro:property name="plate_height" value="1.290"/>
-  <xacro:property name="plate_length" value="0.1"/>
+  <xacro:property name="plate_width" value="0.885" />
+  <xacro:property name="plate_height" value="1.290" />
+  <xacro:property name="plate_length" value="0.1" />
   <link name="fork_plate">
     <visual>
@@ -59,5 +69,5 @@
       <geometry>
         <mesh filename="package://forklift_cpp/models/forklift/meshes/fork_plate_correct_scale.dae"
-        scale="1 1 0.77"
+          scale="1 1 0.77"
         />
       </geometry>
@@ -82,8 +92,12 @@
   <xacro:fork id="1" mass="15" scale="1" fork_attach_offsets="0.05 0.2 -0.35"></xacro:fork>
   <xacro:fork id="2" mass="15" scale="1" fork_attach_offsets="0.05 -0.2 -0.35"></xacro:fork>
-  <xacro:wheel name="right_wheel" mass="5" scale="1" x="0.8" y="-0.4" z="-0.35" yaw="${pi/2}" axis="-1"></xacro:wheel>
-  <xacro:wheel name="right_wheel_back" mass="5" scale="1" x="-0.65" y="-0.4" z="-0.35" yaw="${pi/2}" axis="-1"></xacro:wheel>
-  <xacro:wheel name="left_wheel" mass="5" scale="1" x="0.8" y="0.4" z="-0.35" yaw="-${pi/2}"  axis="-1"></xacro:wheel>
-  <xacro:wheel name="left_wheel_back" mass="5" scale="1" x="-0.65" y="0.4" z="-0.35" yaw="-${pi/2}" axis="-1"></xacro:wheel>
+  <xacro:wheel name="right_wheel" mass="5" scale="1" x="0.8" y="-0.4" z="-0.35" yaw="${pi/2}"
+    axis="-1"></xacro:wheel>
+  <xacro:wheel name="right_wheel_back" mass="5" scale="1" x="-0.65" y="-0.4" z="-0.35" yaw="${pi/2}"
+    axis="-1"></xacro:wheel>
+  <xacro:wheel name="left_wheel" mass="5" scale="1" x="0.8" y="0.4" z="-0.35" yaw="-${pi/2}"
+    axis="-1"></xacro:wheel>
+  <xacro:wheel name="left_wheel_back" mass="5" scale="1" x="-0.65" y="0.4" z="-0.35" yaw="-${pi/2}"
+    axis="-1"></xacro:wheel>
   <gazebo>
     <!--

File: src/forklift_cpp/urdf/wheel.xacro (robot description, xacro)
@@ -1,33 +1,37 @@
 <?xml version="1.0" encoding="UTF-8"?>
+<!--
+  Copyright (c) Elmeri Pohjois-Koivisto
+  See robot.urdf.xacro for licensing
+-->
 <robot xmlns:xacro="http://www.ros.org/wiki/xacro">
-    <xacro:property name="wheel_width" value="0.15" />
-    <xacro:property name="wheel_radius" value="0.25" />
-    <xacro:include filename="inertial_macros.xacro" />
-    <xacro:macro name="wheel" params="name mass scale x y z yaw axis">
-  <joint name="${name}_joint" type="continuous">
-    <parent link="base_link" />
-    <child link="${name}" />
-    <origin xyz="${x} ${y} ${z}" rpy="${pi/2} 0 0" />
-    <axis xyz="0 0 ${axis}" />
-  </joint>
-  <link name="${name}">
-    <visual>
-      <origin xyz="0 0 0" rpy="${yaw} 0 0" />
-      <geometry>
-        <!--The
+  <xacro:property name="wheel_width" value="0.15" />
+  <xacro:property name="wheel_radius" value="0.25" />
+  <xacro:include filename="inertial_macros.xacro" />
+  <xacro:macro name="wheel" params="name mass scale x y z yaw axis">
+    <joint name="${name}_joint" type="continuous">
+      <parent link="base_link" />
+      <child link="${name}" />
+      <origin xyz="${x} ${y} ${z}" rpy="${pi/2} 0 0" />
+      <axis xyz="0 0 ${axis}" />
+    </joint>
+    <link name="${name}">
+      <visual>
+        <origin xyz="0 0 0" rpy="${yaw} 0 0" />
+        <geometry>
+          <!--The
         package resolves into install/forklift_cpp/share/forklift_cpp/-->
-        <mesh filename="package://forklift_cpp/models/forklift/meshes/wheel_correct_scale.dae"/>
-      </geometry>
-    </visual>
-    <collision>
-      <origin xyz="0 0 0" rpy="0 0 0" />
-      <geometry>
-        <cylinder radius="${wheel_radius}" length="${wheel_width}" />
-      </geometry>
-    </collision>
-    <xacro:inertial_cylinder mass="5" radius="${wheel_radius}" length="${wheel_width}">
-      <origin xyz="0 0 0" rpy="0 0 0" />
-    </xacro:inertial_cylinder>
-  </link>
-    </xacro:macro>
+          <mesh filename="package://forklift_cpp/models/forklift/meshes/wheel_correct_scale.dae" />
+        </geometry>
+      </visual>
+      <collision>
+        <origin xyz="0 0 0" rpy="0 0 0" />
+        <geometry>
+          <cylinder radius="${wheel_radius}" length="${wheel_width}" />
+        </geometry>
+      </collision>
+      <xacro:inertial_cylinder mass="5" radius="${wheel_radius}" length="${wheel_width}">
+        <origin xyz="0 0 0" rpy="0 0 0" />
+      </xacro:inertial_cylinder>
+    </link>
+  </xacro:macro>
 </robot>

Commit message: Refactor drop and pickup

File: src/forklift_cpp/urdf/fork.xacro (robot description, xacro)
@@ -29,4 +29,11 @@
       </visual>
       <collision>
+        <gazebo>
+          <surface>
+            <contact>
+              <collide_bitmask>0x01</collide_bitmask>
+            </contact>
+          </surface>
+        </gazebo>
         <origin xyz="0 0 0" rpy="${pi/2} ${pi/2} 0" />
         <geometry>
@@ -67,4 +74,31 @@
       <origin xyz="${fork_length/2} 0 -${fork_attach_height/2-fork_height/2}" rpy="0 0 0" />
     </joint>
+  <gazebo reference="fork_${id}_attach">
+    <collision name="your_collision_name">
+      <surface>
+        <collide_bitmask>0x01</collide_bitmask>
+        <contact>
+          <collide_bitmask>0x01</collide_bitmask>
+        </contact>
+      </surface>
+    </collision>
+</gazebo>
+<gazebo reference="fork_${id}">
+    <collision name="your_collision_name">
+      <surface>
+        <collide_bitmask>0x01</collide_bitmask>
+        <contact>
+          <collide_bitmask>0x01</collide_bitmask>
+        </contact>
+      </surface>
+    </collision>
+</gazebo>
+<gazebo reference="fork_${id}_joint">
+    <preserveFixedJoint>true</preserveFixedJoint>
+  </gazebo>
+  <gazebo reference="fork_attach_${id}_joint">
+    <disableFixedJointLumping>true</disableFixedJointLumping>
+    <preserveFixedJoint>true</preserveFixedJoint>
+  </gazebo>
     <!-- https://osrf-migration.github.io/sdformat-gh-pages/#!/osrf/sdformat/issues/131/page/1-->
   </xacro:macro>

File: src/forklift_cpp/urdf/forklift.urdf.xacro (robot description, xacro)
@@ -159,4 +159,24 @@
   </gazebo>
   -->
+  <gazebo reference="base_link">
+    <collision name="your_collision_name">
+      <surface>
+        <collide_bitmask>0x01</collide_bitmask>
+        <contact>
+          <collide_bitmask>0x01</collide_bitmask>
+        </contact>
+      </surface>
+    </collision>
+</gazebo>
+<gazebo reference="fork_plate">
+    <collision name="your_collision_name">
+      <surface>
+        <collide_bitmask>0x01</collide_bitmask>
+        <contact>
+          <collide_bitmask>0x01</collide_bitmask>
+        </contact>
+      </surface>
+    </collision>
+</gazebo>
   <xacro:plugins namespace="$(arg namespace)"></xacro:plugins>
 </robot>

File: src/forklift_cpp/urdf/forklift_plugins.xacro (robot description, xacro)
@@ -2,13 +2,13 @@
   <xacro:macro name="plugins" params="namespace">
     <gazebo>
-      <!-- <plugin
+      <plugin
       filename="gz-sim-pose-publisher-system"
       name="gz::sim::systems::PosePublisher">
-      <publish_link_pose>true</publish_link_pose>
+      <publish_link_pose>false</publish_link_pose>
       <publish_collision_pose>false</publish_collision_pose>
       <publish_visual_pose>false</publish_visual_pose>
-      <publish_nested_model_pose>false</publish_nested_model_pose>
+      <publish_nested_model_pose>true</publish_nested_model_pose>
       <use_pose_vector_msg>true</use_pose_vector_msg>
-    </plugin> -->
+    </plugin>
       <plugin
         filename="gz-sim-diff-drive-system"
@@ -43,7 +43,16 @@
         <tf_topic>$(arg namespace)/tf</tf_topic>
         <robot_base_frame>base_link</robot_base_frame>
-        <odom_frame>odom</odom_frame>
+        <odom_frame>true_odom</odom_frame>
         <odom_publish_frequency>50</odom_publish_frequency>
     </plugin> -->
+       <plugin filename="gz-sim-detachable-joint-system"
+              name="gz::sim::systems::DetachableJoint">
+       <parent_link>fork_1</parent_link>
+       <child_model>euro_pallet_2</child_model>
+       <child_link>link</child_link>
+       <detach_topic>/euro_pallet_2/detach</detach_topic>
+       <attach_topic>/euro_pallet_2/attach</attach_topic>
+       <output_topic>/euro_pallet_2/state</output_topic>
+      </plugin>
       <plugin filename="gz-sim-joint-state-publisher-system"
         name="gz::sim::systems::JointStatePublisher">

File: src/forklift_cpp/urdf/wheel.xacro (robot description, xacro)
@@ -30,4 +30,14 @@
       </xacro:inertial_cylinder>
     </link>
+    <gazebo reference="${name}">
+    <collision name="your_collision_name">
+      <surface>
+        <collide_bitmask>0x01</collide_bitmask>
+        <contact>
+          <collide_bitmask>0x01</collide_bitmask>
+        </contact>
+      </surface>
+    </collision>
+</gazebo>
   </xacro:macro>
 </robot>
