Commit message: Clean up xacro and add some documentation

File: src/forklift_cpp/urdf/forklift.urdf.xacro (robot description, xacro)
@@ -1,10 +1,9 @@
 <?xml version="1.0"?>
-<robot xmlns:xacro="http://www.ros.org/wiki/xacro">
+<robot xmlns:xacro="http://www.ros.org/wiki/xacro" name="forklift">
+  <xacro:arg name="namespace" default="" />
   <xacro:include filename="inertial_macros.xacro" />
   <xacro:include filename="fork.xacro" />
   <xacro:include filename="wheel.xacro" />
-  <material name="white">
-    <color rgba="1 1 1 1" />
-  </material>
+  <xacro:include filename="forklift_plugins.xacro" />
   <!-- BASE LINK -->
   <xacro:property name="scaler" value="1.0" />
@@ -98,15 +97,4 @@
   <xacro:wheel name="left_wheel_back" mass="5" scale="1" x="-0.65" y="0.4" z="-0.35" yaw="-${pi/2}"
     axis="-1"></xacro:wheel>
-  <gazebo>
-    <!--
-    <plugin filename="gz-sim-touchplugin-system"
-      name="gz::sim::systems::TouchPlugin">
-      <target>cube</target>
-      <time>0.001</time>
-      <enabled>true</enabled>
-     <namespace>$(arg namespace)</namespace>
-    </plugin>
-  -->
-  </gazebo>
   <gazebo reference="fork_plate">
     <sensor name='sensor_contact' type='contact'>
@@ -171,3 +159,4 @@
   </gazebo>
   -->
+  <xacro:plugins namespace="$(arg namespace)"></xacro:plugins>
 </robot>

Commit message: Start refactoring attach

File: src/forklift_cpp/urdf/forklift.urdf.xacro (robot description, xacro)
@@ -85,5 +85,5 @@
     <origin xyz="1.15 0 0.025" rpy="0 0 0" />
     <axis xyz="0 0 1" />
-    <limit effort="2500" lower="0.0" upper="5.0" velocity="0.5" />
+    <limit effort="2500" lower="0.0" upper="2.0" velocity="0.5" />
   </joint>
   <xacro:fork id="1" mass="15" scale="1" fork_attach_offsets="0.05 0.2 -0.35"></xacro:fork>

File: src/forklift_cpp/urdf/forklift_plugins.xacro (robot description, xacro)
@@ -51,7 +51,7 @@
        <child_model>euro_pallet_2</child_model>
        <child_link>link</child_link>
-       <detach_topic>/euro_pallet_2/detach</detach_topic>
-       <attach_topic>/euro_pallet_2/attach</attach_topic>
-       <output_topic>/euro_pallet_2/state</output_topic>
+       <detach_topic>${namespace}/euro_pallet_2/detach</detach_topic>
+       <attach_topic>${namespace}/euro_pallet_2/attach</attach_topic>
+       <output_topic>${namespace}/euro_pallet_2/state</output_topic>
       </plugin>
       <plugin filename="gz-sim-joint-state-publisher-system"
